Commit message: finished assignment 5

File: body.urdf (robot description, URDF)
Before this commit: robot robot, 9 links, 8 joints
Links:
- removed link LeftLeg
- removed link LeftLowerLeg
- link BackLeg: geometry collision box size=0.2 0.2 0.2; visual box size=0.2 0.2 0.2
- link BackLowerLeg: geometry collision box size=0.2 1 0.2; visual box size=0.2 1 0.2
- link FrontLeg: geometry collision box size=0.2 0.2 0.2; visual box size=0.2 0.2 0.2
- link FrontLowerLeg: geometry collision box size=0.2 1 0.2; visual box size=0.2 1 0.2
Joints:
- removed joint LeftLeg_LeftLowerLeg
- removed joint Torso_LeftLeg
- joint BackLeg_BackLowerLeg: axis 1 0 0 -> 0 0 1; origin xyz=0 -1 0 rpy=0 0 0 -> xyz=0 -0.2 0 rpy=0 0 0
- joint FrontLeg_FrontLowerLeg: axis 1 0 0 -> 0 0 1; origin xyz=0 1 0 rpy=0 0 0 -> xyz=0 0.2 0 rpy=0 0 0
- joint Torso_BackLeg: axis 1 0 0 -> 0 0 1; origin xyz=0 -0.5 1 rpy=0 0 0 -> xyz=0 -0.5 0.6 rpy=0 0 0
- joint Torso_FrontLeg: axis 1 0 0 -> 0 0 1; origin xyz=0 0.5 1 rpy=0 0 0 -> xyz=0 0.5 0.6 rpy=0 0 0

Commit message: sike, now i finished it

File: body.urdf (robot description, URDF)
Before this commit: robot robot, 7 links, 6 joints
Links:
- removed link RightLeg
- removed link RightLowerLeg
Joints:
- removed joint RightLeg_RightLowerLeg
- removed joint Torso_RightLeg

Commit message: got the beginning down

File: body.urdf (robot description, URDF)
Before this commit: robot robot, 5 links, 4 joints
Links:
- removed link BackLowerLeg
- removed link FrontLeg
- removed link FrontLowerLeg
- link BackLeg: geometry collision box size=1.7692563495036213 0.7281819643251011 0.7764790329310851; visual box size=1.7692563495036213 0.7281819643251011 0.7764790329310851
- link Torso: geometry collision box size=1.9431422197268422 1 1; visual box size=1.9431422197268422 1 1
Joints:
- removed joint BackLeg_BackLowerLeg
- removed joint FrontLeg_FrontLowerLeg
- removed joint Torso_FrontLeg
- joint Torso_BackLeg: origin xyz=0 -0.5 0.6 rpy=0 0 0 -> xyz=-3.028428890136579 0 3 rpy=0 0 0

Commit message: got the color of the links to change

File: body.urdf (robot description, URDF)
Before this commit: robot robot, 2 links, 1 joints
Links:
- removed link BackLeg
- added link Apple, mass 1; collision box size=1.8982656594156493 1.6199428530301592 1.6978296615022679; visual box size=1.8982656594156493 1.6199428530301592 1.6978296615022679
- added link Dog, mass 1; collision box size=1.8190262148970529 1.8408563019091235 1.6351405577286517; visual box size=1.8190262148970529 1.8408563019091235 1.6351405577286517
- added link Flower, mass 1; collision box size=0.5082072090082435 1.1966199886972309 0.1029873141636104; visual box size=0.5082072090082435 1.1966199886972309 0.1029873141636104
- added link Fox, mass 1; collision box size=1.4108517441192179 1.5693483141416869 0.4410662357597346; visual box size=1.4108517441192179 1.5693483141416869 0.4410662357597346
- added link Person, mass 1; collision box size=1.3583436339011163 0.8174025703025032 0.8983262822016593; visual box size=1.3583436339011163 0.8174025703025032 0.8983262822016593
- link Torso: geometry collision box size=1.1340697227591712 1 1; visual box size=1.1340697227591712 1 1
Joints:
- removed joint Torso_BackLeg
- added joint Apple_Dog: type revolute, parent Apple, child Dog, origin xyz=1.8982656594156493 0 0 rpy=0 0 0, axis 0 1 0, limit lower=-3.14159 upper=3.14159 effort=0.0 velocity=0.0
- added joint Dog_Person: type revolute, parent Dog, child Person, origin xyz=1.8190262148970529 0 0 rpy=0 0 0, axis 0 1 0, limit lower=-3.14159 upper=3.14159 effort=0.0 velocity=0.0
- added joint Fox_Flower: type revolute, parent Fox, child Flower, origin xyz=1.4108517441192179 0 0 rpy=0 0 0, axis 0 1 0, limit lower=-3.14159 upper=3.14159 effort=0.0 velocity=0.0
- added joint Person_Fox: type revolute, parent Person, child Fox, origin xyz=1.3583436339011163 0 0 rpy=0 0 0, axis 0 1 0, limit lower=-3.14159 upper=3.14159 effort=0.0 velocity=0.0
- added joint Torso_Apple: type revolute, parent Torso, child Apple, origin xyz=-3.4329651386204145 0 3 rpy=0 0 0, axis 0 1 0, limit lower=-3.14159 upper=3.14159 effort=0.0 velocity=0.0

Commit message: edited readme

File: body.urdf (robot description, URDF)
Before this commit: robot robot, 6 links, 5 joints
Links:
- added link Neighbor, mass 1; collision box size=0.6876249704557662 1.4320532730767603 1.8527390029480306; visual box size=0.6876249704557662 1.4320532730767603 1.8527390029480306
- link Apple: geometry collision box size=0.1485445421829008 0.6617292029600665 0.42742430245794183; visual box size=0.1485445421829008 0.6617292029600665 0.42742430245794183
- link Dog: geometry collision box size=0.7002599552787523 0.8365126594946617 1.3845129823572069; visual box size=0.7002599552787523 0.8365126594946617 1.3845129823572069
- link Flower: geometry collision box size=1.844269304943553 1.5492373680667257 0.6911105154509176; visual box size=1.844269304943553 1.5492373680667257 0.6911105154509176
- link Fox: geometry collision box size=1.0472935529470797 1.9779950298311053 0.08260588545919045; visual box size=1.0472935529470797 1.9779950298311053 0.08260588545919045
- link Person: geometry collision box size=1.4545903679864824 0.7471339979944409 0.9185690685772914; visual box size=1.4545903679864824 0.7471339979944409 0.9185690685772914
- link Torso: geometry collision box size=1.7573159603520403 1 1; visual box size=1.7573159603520403 1 1
Joints:
- added joint Flower_Neighbor: type revolute, parent Flower, child Neighbor, origin xyz=1.844269304943553 0 0 rpy=0 0 0, axis 0 1 0, limit lower=-3.14159 upper=3.14159 effort=0.0 velocity=0.0
- joint Apple_Dog: origin xyz=1.8982656594156493 0 0 rpy=0 0 0 -> xyz=0.1485445421829008 0 0 rpy=0 0 0
- joint Dog_Person: origin xyz=1.8190262148970529 0 0 rpy=0 0 0 -> xyz=0.7002599552787523 0 0 rpy=0 0 0
- joint Fox_Flower: origin xyz=1.4108517441192179 0 0 rpy=0 0 0 -> xyz=1.0472935529470797 0 0 rpy=0 0 0
- joint Person_Fox: origin xyz=1.3583436339011163 0 0 rpy=0 0 0 -> xyz=1.4545903679864824 0 0 rpy=0 0 0
- joint Torso_Apple: origin xyz=-3.4329651386204145 0 3 rpy=0 0 0 -> xyz=1.8786579801760201 0 3 rpy=0 0 0

Commit message: got rid of side panels in the visual

File: body.urdf (robot description, URDF)
Before this commit: robot robot, 7 links, 6 joints
Links:
- added link Coffee, mass 1; collision box size=0.46600503881880995 1.3144505152611807 1.7584620044147339; visual box size=0.46600503881880995 1.3144505152611807 1.7584620044147339
- link Apple: geometry collision box size=1.5484594630608413 0.10547728106503129 1.2840350188108556; visual box size=1.5484594630608413 0.10547728106503129 1.2840350188108556
- link Dog: geometry collision box size=0.077704677919473 1.9113699971109968 0.4115862454085284; visual box size=0.077704677919473 1.9113699971109968 0.4115862454085284
- link Flower: geometry collision box size=1.0530296882102124 0.8761855061743382 1.393009351659914; visual box size=1.0530296882102124 0.8761855061743382 1.393009351659914
- link Fox: geometry collision box size=0.4901626951711886 1.42579429715745 0.6253533667884623; visual box size=0.4901626951711886 1.42579429715745 0.6253533667884623
- link Neighbor: geometry collision box size=1.863216431746603 0.3053266239894876 0.6852136294179394; visual box size=1.863216431746603 0.3053266239894876 0.6852136294179394
- link Person: geometry collision box size=0.9299617385812589 0.2309725123194224 1.9970964847245363; visual box size=0.9299617385812589 0.2309725123194224 1.9970964847245363
- link Torso: geometry collision box size=0.1339647526360388 1 1; visual box size=0.1339647526360388 1 1
Joints:
- added joint Neighbor_Coffee: type revolute, parent Neighbor, child Coffee, origin xyz=1.863216431746603 0 0 rpy=0 0 0, axis 0 1 0, limit lower=-3.14159 upper=3.14159 effort=0.0 velocity=0.0
- joint Apple_Dog: origin xyz=0.1485445421829008 0 0 rpy=0 0 0 -> xyz=1.5484594630608413 0 0 rpy=0 0 0
- joint Dog_Person: origin xyz=0.7002599552787523 0 0 rpy=0 0 0 -> xyz=0.077704677919473 0 0 rpy=0 0 0
- joint Flower_Neighbor: origin xyz=1.844269304943553 0 0 rpy=0 0 0 -> xyz=1.0530296882102124 0 0 rpy=0 0 0
- joint Fox_Flower: origin xyz=1.0472935529470797 0 0 rpy=0 0 0 -> xyz=0.4901626951711886 0 0 rpy=0 0 0
- joint Person_Fox: origin xyz=1.4545903679864824 0 0 rpy=0 0 0 -> xyz=0.9299617385812589 0 0 rpy=0 0 0
- joint Torso_Apple: origin xyz=1.8786579801760201 0 3 rpy=0 0 0 -> xyz=-0.9330176236819806 0 3 rpy=0 0 0

Commit message: gonna start again on try1

File: body.urdf (robot description, URDF)
Before this commit: robot robot, 8 links, 7 joints
Links:
- added link A, mass 1; collision box size=0.7569521484359374 -3.887011760518811 -3.099818727875463; visual box size=0.7569521484359374 -3.887011760518811 -3.099818727875463
- added link Algebra, mass 1; collision box size=-1.3712361893478233 0.6379765606436134 0.08682019578652866; visual box size=-1.3712361893478233 0.6379765606436134 0.08682019578652866
- added link Artifact, mass 1; collision box size=-0.8757980087837662 3.963980932938089 0.48982509640878646; visual box size=-0.8757980087837662 3.963980932938089 0.48982509640878646
- added link Bottle, mass 1; collision box size=3.62885842959487 0.7651285527498688 -0.8948418280035124; visual box size=3.62885842959487 0.7651285527498688 -0.8948418280035124
- added link Chair, mass 1; collision box size=3.96547839886556 -2.9181206135810127 3.148876409451346; visual box size=3.96547839886556 -2.9181206135810127 3.148876409451346
- added link Clock, mass 1; collision box size=2.0618391444296877 3.5724016053634253 1.4183328836642382; visual box size=2.0618391444296877 3.5724016053634253 1.4183328836642382
- added link Code, mass 1; collision box size=0.9047262112199759 -1.144441018463172 -0.7279416338677187; visual box size=0.9047262112199759 -1.144441018463172 -0.7279416338677187
- added link Computer, mass 1; collision box size=0.5301697276604163 0.8440334645579322 3.143060515351383; visual box size=0.5301697276604163 0.8440334645579322 3.143060515351383
- added link Construct, mass 1; collision box size=-3.6088456911890026 2.2916669345044154 -2.8173024654362413; visual box size=-3.6088456911890026 2.2916669345044154 -2.8173024654362413
- added link Cracking, mass 1; collision box size=3.183172129077236 -2.0636915024321105 -2.7988783868013964; visual box size=3.183172129077236 -2.0636915024321105 -2.7988783868013964
- added link Feature, mass 1; collision box size=-2.544978316926925 -3.0942495071298772 -0.2959398946735865; visual box size=-2.544978316926925 -3.0942495071298772 -0.2959398946735865
- added link Flute, mass 1; collision box size=-2.0884603681142657 1.7371392925765203 3.352001768209174; visual box size=-2.0884603681142657 1.7371392925765203 3.352001768209174
- added link Garbage, mass 1; collision box size=-2.1294498826769113 1.8910444087128937 3.5600773524581246; visual box size=-2.1294498826769113 1.8910444087128937 3.5600773524581246
- added link Genshin, mass 1; collision box size=2.8497242912203973 1.7153188241435302 3.3525399536828333; visual box size=2.8497242912203973 1.7153188241435302 3.3525399536828333
- added link Impact, mass 1; collision box size=-1.4210140652549423 -3.32730608098017 -1.165311054865743; visual box size=-1.4210140652549423 -3.32730608098017 -1.165311054865743
- added link Interview, mass 1; collision box size=1.8612030870073468 -3.7948028785332975 3.2709535450768774; visual box size=1.8612030870073468 -3.7948028785332975 3.2709535450768774
- added link Lamp, mass 1; collision box size=-2.9981954638586634 -1.8334577700647152 -1.8931743627700168; visual box size=-2.9981954638586634 -1.8334577700647152 -1.8931743627700168
- added link Library, mass 1; collision box size=-3.478408600993257 -1.3572376402765318 -0.6429488367093228; visual box size=-3.478408600993257 -1.3572376402765318 -0.6429488367093228
- added link Linear, mass 1; collision box size=3.1055716814480583 -2.7532857597298186 0.029684376366704512; visual box size=3.1055716814480583 -2.7532857597298186 0.029684376366704512
- added link Mana, mass 1; collision box size=0.28509231386112344 1.749364127922771 0.48656341197487674; visual box size=0.28509231386112344 1.749364127922771 0.48656341197487674
- added link Perspective, mass 1; collision box size=3.595696210952716 1.3824494702998011 -1.0275304730167028; visual box size=3.595696210952716 1.3824494702998011 -1.0275304730167028
- added link Phone, mass 1; collision box size=-2.8880074255433525 3.372902802116145 -0.48724870433689293; visual box size=-2.8880074255433525 3.372902802116145 -0.48724870433689293
- added link Pound, mass 1; collision box size=-3.033421548854947 -3.0394761764351834 -3.158913436822748; visual box size=-3.033421548854947 -3.0394761764351834 -3.158913436822748
- added link Powerade, mass 1; collision box size=-2.3828213532729485 -3.5422560560233007 -1.3078279093767389; visual box size=-2.3828213532729485 -3.5422560560233007 -1.3078279093767389
- added link Programmer, mass 1; collision box size=-0.8116291273060554 -3.6826204109815714 1.4462331898883214; visual box size=-0.8116291273060554 -3.6826204109815714 1.4462331898883214
- added link Shuffle, mass 1; collision box size=3.100761422111723 0.786921881168225 -2.439550727278034; visual box size=3.100761422111723 0.786921881168225 -2.439550727278034
- added link Stool, mass 1; collision box size=0.25200751326674276 -0.8772865235311009 -1.369155277160183; visual box size=0.25200751326674276 -0.8772865235311009 -1.369155277160183
- added link Systems, mass 1; collision box size=-0.86095353395367 -2.326725464037974 -0.2187538285606223; visual box size=-0.86095353395367 -2.326725464037974 -0.2187538285606223
- added link Table, mass 1; collision box size=-1.1917414902798837 -3.884912688241041 -1.7955488080051705; visual box size=-1.1917414902798837 -3.884912688241041 -1.7955488080051705
- added link The, mass 1; collision box size=3.070035704204644 0.1900647308215726 0.2095606711977105; visual box size=3.070035704204644 0.1900647308215726 0.2095606711977105
- added link Token, mass 1; collision box size=1.2147329976717893 -0.1540520270965633 -2.3716358002081854; visual box size=1.2147329976717893 -0.1540520270965633 -2.3716358002081854
- added link Top, mass 1; collision box size=0.9793192091908001 -1.5101766716985798 -0.7435355871159199; visual box size=0.9793192091908001 -1.5101766716985798 -0.7435355871159199
- added link Water, mass 1; collision box size=1.236335462597994 3.5272861523285286 -2.0301973484753484; visual box size=1.236335462597994 3.5272861523285286 -2.0301973484753484
- link Apple: geometry collision box size=0.8468485769730447 0.982875023222024 1.3441747900163272; visual box size=0.8468485769730447 0.982875023222024 1.3441747900163272
- link Coffee: geometry collision box size=-2.9307432124667665 -0.22120995925897446 -1.7968048503773222; visual box size=-2.9307432124667665 -0.22120995925897446 -1.7968048503773222
- link Dog: geometry collision box size=-1.5329442998018896 0.8851597940525844 -0.741285107797542; visual box size=-1.5329442998018896 0.8851597940525844 -0.741285107797542
- link Flower: geometry collision box size=-2.302376526293619 3.6766701528403285 3.0061669338016115; visual box size=-2.302376526293619 3.6766701528403285 3.0061669338016115
- link Fox: geometry collision box size=-3.4856232938115097 1.8697551513649024 -1.4836741053451785; visual box size=-3.4856232938115097 1.8697551513649024 -1.4836741053451785
- link Neighbor: geometry collision box size=-1.7631489405726954 -1.296090683026069 2.237631969897264; visual box size=-1.7631489405726954 -1.296090683026069 2.237631969897264
- link Person: geometry collision box size=2.0367400244093385 -0.9377300729356239 -2.9675383243653304; visual box size=2.0367400244093385 -0.9377300729356239 -2.9675383243653304
- link Torso: geometry collision box size=1.2430720868493048 1 1; visual box size=1.2430720868493048 1 1
Joints:
- added joint A_Programmer: type revolute, parent A, child Programmer, origin xyz=0.7569521484359374 0 0 rpy=0 0 0, axis 0 1 0, limit lower=-3.14159 upper=3.14159 effort=0.0 velocity=0.0
- added joint Artifact_Feature: type revolute, parent Artifact, child Feature, origin xyz=-0.8757980087837662 0 0 rpy=0 0 0, axis 0 1 0, limit lower=-3.14159 upper=3.14159 effort=0.0 velocity=0.0
- added joint Bottle_Clock: type revolute, parent Bottle, child Clock, origin xyz=3.62885842959487 0 0 rpy=0 0 0, axis 0 1 0, limit lower=-3.14159 upper=3.14159 effort=0.0 velocity=0.0
- added joint Chair_Stool: type revolute, parent Chair, child Stool, origin xyz=3.96547839886556 0 0 rpy=0 0 0, axis 0 1 0, limit lower=-3.14159 upper=3.14159 effort=0.0 velocity=0.0
- added joint Clock_Lamp: type revolute, parent Clock, child Lamp, origin xyz=2.0618391444296877 0 0 rpy=0 0 0, axis 0 1 0, limit lower=-3.14159 upper=3.14159 effort=0.0 velocity=0.0
- added joint Code_Interview: type revolute, parent Code, child Interview, origin xyz=0.9047262112199759 0 0 rpy=0 0 0, axis 0 1 0, limit lower=-3.14159 upper=3.14159 effort=0.0 velocity=0.0
- added joint Coffee_Phone: type revolute, parent Coffee, child Phone, origin xyz=-2.9307432124667665 0 0 rpy=0 0 0, axis 0 1 0, limit lower=-3.14159 upper=3.14159 effort=0.0 velocity=0.0
- added joint Computer_Bottle: type revolute, parent Computer, child Bottle, origin xyz=0.5301697276604163 0 0 rpy=0 0 0, axis 0 1 0, limit lower=-3.14159 upper=3.14159 effort=0.0 velocity=0.0
- added joint Construct_Artifact: type revolute, parent Construct, child Artifact, origin xyz=-3.6088456911890026 0 0 rpy=0 0 0, axis 0 1 0, limit lower=-3.14159 upper=3.14159 effort=0.0 velocity=0.0
- added joint Cracking_The: type revolute, parent Cracking, child The, origin xyz=3.183172129077236 0 0 rpy=0 0 0, axis 0 1 0, limit lower=-3.14159 upper=3.14159 effort=0.0 velocity=0.0
- added joint Feature_Token: type revolute, parent Feature, child Token, origin xyz=-2.544978316926925 0 0 rpy=0 0 0, axis 0 1 0, limit lower=-3.14159 upper=3.14159 effort=0.0 velocity=0.0
- added joint Flute_Garbage: type revolute, parent Flute, child Garbage, origin xyz=-2.0884603681142657 0 0 rpy=0 0 0, axis 0 1 0, limit lower=-3.14159 upper=3.14159 effort=0.0 velocity=0.0
- added joint Garbage_Powerade: type revolute, parent Garbage, child Powerade, origin xyz=-2.1294498826769113 0 0 rpy=0 0 0, axis 0 1 0, limit lower=-3.14159 upper=3.14159 effort=0.0 velocity=0.0
- added joint Genshin_Flute: type revolute, parent Genshin, child Flute, origin xyz=2.8497242912203973 0 0 rpy=0 0 0, axis 0 1 0, limit lower=-3.14159 upper=3.14159 effort=0.0 velocity=0.0
- added joint Impact_Genshin: type revolute, parent Impact, child Genshin, origin xyz=-1.4210140652549423 0 0 rpy=0 0 0, axis 0 1 0, limit lower=-3.14159 upper=3.14159 effort=0.0 velocity=0.0
- added joint Interview_Linear: type revolute, parent Interview, child Linear, origin xyz=1.8612030870073468 0 0 rpy=0 0 0, axis 0 1 0, limit lower=-3.14159 upper=3.14159 effort=0.0 velocity=0.0
- added joint Lamp_Systems: type revolute, parent Lamp, child Systems, origin xyz=-2.9981954638586634 0 0 rpy=0 0 0, axis 0 1 0, limit lower=-3.14159 upper=3.14159 effort=0.0 velocity=0.0
- added joint Library_Mana: type revolute, parent Library, child Mana, origin xyz=-3.478408600993257 0 0 rpy=0 0 0, axis 0 1 0, limit lower=-3.14159 upper=3.14159 effort=0.0 velocity=0.0
- added joint Linear_Algebra: type revolute, parent Linear, child Algebra, origin xyz=3.1055716814480583 0 0 rpy=0 0 0, axis 0 1 0, limit lower=-3.14159 upper=3.14159 effort=0.0 velocity=0.0
- added joint Mana_Top: type revolute, parent Mana, child Top, origin xyz=0.28509231386112344 0 0 rpy=0 0 0, axis 0 1 0, limit lower=-3.14159 upper=3.14159 effort=0.0 velocity=0.0
- added joint Perspective_Cracking: type revolute, parent Perspective, child Cracking, origin xyz=3.595696210952716 0 0 rpy=0 0 0, axis 0 1 0, limit lower=-3.14159 upper=3.14159 effort=0.0 velocity=0.0
- added joint Phone_Table: type revolute, parent Phone, child Table, origin xyz=-2.8880074255433525 0 0 rpy=0 0 0, axis 0 1 0, limit lower=-3.14159 upper=3.14159 effort=0.0 velocity=0.0
- added joint Pound_Computer: type revolute, parent Pound, child Computer, origin xyz=-3.033421548854947 0 0 rpy=0 0 0, axis 0 1 0, limit lower=-3.14159 upper=3.14159 effort=0.0 velocity=0.0
- added joint Powerade_Construct: type revolute, parent Powerade, child Construct, origin xyz=-2.3828213532729485 0 0 rpy=0 0 0, axis 0 1 0, limit lower=-3.14159 upper=3.14159 effort=0.0 velocity=0.0
- added joint Programmer_Perspective: type revolute, parent Programmer, child Perspective, origin xyz=-0.8116291273060554 0 0 rpy=0 0 0, axis 0 1 0, limit lower=-3.14159 upper=3.14159 effort=0.0 velocity=0.0
- added joint Shuffle_Chair: type revolute, parent Shuffle, child Chair, origin xyz=3.100761422111723 0 0 rpy=0 0 0, axis 0 1 0, limit lower=-3.14159 upper=3.14159 effort=0.0 velocity=0.0
- added joint Stool_Water: type revolute, parent Stool, child Water, origin xyz=0.25200751326674276 0 0 rpy=0 0 0, axis 0 1 0, limit lower=-3.14159 upper=3.14159 effort=0.0 velocity=0.0
- added joint Systems_A: type revolute, parent Systems, child A, origin xyz=-0.86095353395367 0 0 rpy=0 0 0, axis 0 1 0, limit lower=-3.14159 upper=3.14159 effort=0.0 velocity=0.0
- added joint Table_Impact: type revolute, parent Table, child Impact, origin xyz=-1.1917414902798837 0 0 rpy=0 0 0, axis 0 1 0, limit lower=-3.14159 upper=3.14159 effort=0.0 velocity=0.0
- added joint The_Code: type revolute, parent The, child Code, origin xyz=3.070035704204644 0 0 rpy=0 0 0, axis 0 1 0, limit lower=-3.14159 upper=3.14159 effort=0.0 velocity=0.0
- added joint Token_Library: type revolute, parent Token, child Library, origin xyz=1.2147329976717893 0 0 rpy=0 0 0, axis 0 1 0, limit lower=-3.14159 upper=3.14159 effort=0.0 velocity=0.0
- added joint Top_Shuffle: type revolute, parent Top, child Shuffle, origin xyz=0.9793192091908001 0 0 rpy=0 0 0, axis 0 1 0, limit lower=-3.14159 upper=3.14159 effort=0.0 velocity=0.0
- added joint Water_Pound: type revolute, parent Water, child Pound, origin xyz=1.236335462597994 0 0 rpy=0 0 0, axis 0 1 0, limit lower=-3.14159 upper=3.14159 effort=0.0 velocity=0.0
- joint Apple_Dog: origin xyz=1.5484594630608413 0 0 rpy=0 0 0 -> xyz=0.8468485769730447 0 0 rpy=0 0 0
- joint Dog_Person: origin xyz=0.077704677919473 0 0 rpy=0 0 0 -> xyz=-1.5329442998018896 0 0 rpy=0 0 0
- joint Flower_Neighbor: origin xyz=1.0530296882102124 0 0 rpy=0 0 0 -> xyz=-2.302376526293619 0 0 rpy=0 0 0
- joint Fox_Flower: origin xyz=0.4901626951711886 0 0 rpy=0 0 0 -> xyz=-3.4856232938115097 0 0 rpy=0 0 0
- joint Neighbor_Coffee: origin xyz=1.863216431746603 0 0 rpy=0 0 0 -> xyz=-1.7631489405726954 0 0 rpy=0 0 0
- joint Person_Fox: origin xyz=0.9299617385812589 0 0 rpy=0 0 0 -> xyz=2.0367400244093385 0 0 rpy=0 0 0
- joint Torso_Apple: origin xyz=-0.9330176236819806 0 3 rpy=0 0 0 -> xyz=1.6215360434246524 -4 0 rpy=0 0 0
