Commit message: the joints look weird

File: body.urdf (robot description, URDF)
Before this commit: robot robot, 8 links, 7 joints
Links:
- added link Flute, mass 1; collision box size=1.3026705945118322 1.274122703003618 0.9579544851806365; visual box size=1.3026705945118322 1.274122703003618 0.9579544851806365
- added link Garbage, mass 1; collision box size=0.26556302114630004 0.5089038672914352 1.9043754774100123; visual box size=0.26556302114630004 0.5089038672914352 1.9043754774100123
- added link Genshin, mass 1; collision box size=1.899371955289446 0.5084493776183792 1.6746158129698527; visual box size=1.899371955289446 0.5084493776183792 1.6746158129698527
- added link Impact, mass 1; collision box size=1.0529488010819283 0.4957528563726159 0.3408329575943234; visual box size=1.0529488010819283 0.4957528563726159 0.3408329575943234
- added link Phone, mass 1; collision box size=0.9306896762716967 0.9384648878677972 1.8494877436020039; visual box size=0.9306896762716967 0.9384648878677972 1.8494877436020039
- added link Powerade, mass 1; collision box size=1.948124591401348 0.6997496669148984 0.9916896507148016; visual box size=1.948124591401348 0.6997496669148984 0.9916896507148016
- added link Table, mass 1; collision box size=1.9634252835986936 1.4465410521426378 1.424903850281021; visual box size=1.9634252835986936 1.4465410521426378 1.424903850281021
- added link construct, mass 1; collision box size=0.1400899398231643 0.0007257362514021537 0.11362913368740646; visual box size=0.1400899398231643 0.0007257362514021537 0.11362913368740646
- link Apple: geometry collision box size=0.287963969254895 1.7908743854822007 0.045409789018527213; visual box size=0.287963969254895 1.7908743854822007 0.045409789018527213
- link Coffee: geometry collision box size=0.38963946752698075 0.876419911703926 0.6558792428411186; visual box size=0.38963946752698075 0.876419911703926 0.6558792428411186
- link Dog: geometry collision box size=0.03518901717214562 0.6297635215514472 0.40362017826042673; visual box size=0.03518901717214562 0.6297635215514472 0.40362017826042673
- link Flower: geometry collision box size=1.4669235270929977 0.5336396436843207 0.7183889194305815; visual box size=1.4669235270929977 0.5336396436843207 0.7183889194305815
- link Fox: geometry collision box size=0.8623580345477688 0.12399584576510847 0.583055569214415; visual box size=0.8623580345477688 0.12399584576510847 0.583055569214415
- link Neighbor: geometry collision box size=0.5353439014755232 1.6505978599657716 0.44042075056824603; visual box size=0.5353439014755232 1.6505978599657716 0.44042075056824603
- link Person: geometry collision box size=1.9475532620031302 0.4529948662413974 0.04265430149831695; visual box size=1.9475532620031302 0.4529948662413974 0.04265430149831695
- link Torso: geometry collision box size=0.1545777136139488 1 1; visual box size=0.1545777136139488 1 1
Joints:
- added joint Coffee_Phone: type revolute, parent Coffee, child Phone, origin xyz=0 0.9384648878677972 0 rpy=0 0 0, axis 0 1 0, limit lower=-3.14159 upper=3.14159 effort=0.0 velocity=0.0
- added joint Flute_Garbage: type revolute, parent Flute, child Garbage, origin xyz=0.26556302114630004 0 0 rpy=0 0 0, axis 0 1 0, limit lower=-3.14159 upper=3.14159 effort=0.0 velocity=0.0
- added joint Garbage_Powerade: type revolute, parent Garbage, child Powerade, origin xyz=0 0.6997496669148984 0 rpy=0 0 0, axis 0 1 0, limit lower=-3.14159 upper=3.14159 effort=0.0 velocity=0.0
- added joint Genshin_Flute: type revolute, parent Genshin, child Flute, origin xyz=0 1.274122703003618 0 rpy=0 0 0, axis 0 1 0, limit lower=-3.14159 upper=3.14159 effort=0.0 velocity=0.0
- added joint Impact_Genshin: type revolute, parent Impact, child Genshin, origin xyz=1.899371955289446 0 0 rpy=0 0 0, axis 0 1 0, limit lower=-3.14159 upper=3.14159 effort=0.0 velocity=0.0
- added joint Phone_Table: type revolute, parent Phone, child Table, origin xyz=1.9634252835986936 0 0 rpy=0 0 0, axis 0 1 0, limit lower=-3.14159 upper=3.14159 effort=0.0 velocity=0.0
- added joint Powerade_construct: type revolute, parent Powerade, child construct, origin xyz=0.1400899398231643 0 0 rpy=0 0 0, axis 0 1 0, limit lower=-3.14159 upper=3.14159 effort=0.0 velocity=0.0
- added joint Table_Impact: type revolute, parent Table, child Impact, origin xyz=0 0.4957528563726159 0 rpy=0 0 0, axis 0 1 0, limit lower=-3.14159 upper=3.14159 effort=0.0 velocity=0.0
- joint Apple_Dog: origin xyz=1.5484594630608413 0 0 rpy=0 0 0 -> xyz=0.6297635215514472 0 0 rpy=0 0 0
- joint Dog_Person: origin xyz=0.077704677919473 0 0 rpy=0 0 0 -> xyz=1.9475532620031302 0 0 rpy=0 0 0
- joint Flower_Neighbor: origin xyz=1.0530296882102124 0 0 rpy=0 0 0 -> xyz=0 1.6505978599657716 0 rpy=0 0 0
- joint Fox_Flower: origin xyz=0.4901626951711886 0 0 rpy=0 0 0 -> xyz=1.4669235270929977 0 0 rpy=0 0 0
- joint Neighbor_Coffee: origin xyz=1.863216431746603 0 0 rpy=0 0 0 -> xyz=0.38963946752698075 0 0 rpy=0 0 0
- joint Person_Fox: origin xyz=0.9299617385812589 0 0 rpy=0 0 0 -> xyz=0 0.12399584576510847 0 rpy=0 0 0
- joint Torso_Apple: origin xyz=-0.9330176236819806 0 3 rpy=0 0 0 -> xyz=1.0772888568069745 0 3 rpy=0 0 0

Commit message: the joints are kinda messed up

File: body.urdf (robot description, URDF)
Before this commit: robot robot, 16 links, 15 joints
Links:
- removed link Flute
- removed link Garbage
- removed link Powerade
- removed link construct
- link Apple: geometry collision box size=1.9758451444312737 0.7809828042991716 0.000347477689554454; visual box size=1.9758451444312737 0.7809828042991716 0.000347477689554454
- link Coffee: geometry collision box size=0.2483548304608989 1.516369125483459 1.792916509282243; visual box size=0.2483548304608989 1.516369125483459 1.792916509282243
- link Dog: geometry collision box size=1.7793935510854917 1.8726193056021712 1.419733787652017; visual box size=1.7793935510854917 1.8726193056021712 1.419733787652017
- link Flower: geometry collision box size=1.9237069094660273 0.702788051714692 1.6443974403011163; visual box size=1.9237069094660273 0.702788051714692 1.6443974403011163
- link Fox: geometry collision box size=0.1674106681546954 1.315677321488007 1.7006994955676626; visual box size=0.1674106681546954 1.315677321488007 1.7006994955676626
- link Genshin: geometry collision box size=0.8784323146098854 1.3632424817118134 0.8628450814747202; visual box size=0.8784323146098854 1.3632424817118134 0.8628450814747202
- link Impact: geometry collision box size=1.9615455878601433 1.11423884587598 1.41247026036155; visual box size=1.9615455878601433 1.11423884587598 1.41247026036155
- link Neighbor: geometry collision box size=0.009127086097822756 1.7507431506127518 1.0526104673129784; visual box size=0.009127086097822756 1.7507431506127518 1.0526104673129784
- link Person: geometry collision box size=0.6347503224792679 1.4977907160713089 0.8437743315989388; visual box size=0.6347503224792679 1.4977907160713089 0.8437743315989388
- link Phone: geometry collision box size=1.3292760061663584 1.4875272501752297 1.5706954369077708; visual box size=1.3292760061663584 1.4875272501752297 1.5706954369077708
- link Table: geometry collision box size=1.9343168316300634 0.4461966238085431 1.991550672665372; visual box size=1.9343168316300634 0.4461966238085431 1.991550672665372
- link Torso: geometry collision box size=1.2194935760659822 1 1; visual box size=1.2194935760659822 1 1
Joints:
- removed joint Flute_Garbage
- removed joint Garbage_Powerade
- removed joint Genshin_Flute
- removed joint Powerade_construct
- joint Apple_Dog: origin xyz=0.6297635215514472 0 0 rpy=0 0 0 -> xyz=1.9758451444312737 0 0 rpy=0 0 0
- joint Coffee_Phone: origin xyz=0 0.9384648878677972 0 rpy=0 0 0 -> xyz=0 0 0.8964582546411215 rpy=0 0 0
- joint Dog_Person: origin xyz=1.9475532620031302 0 0 rpy=0 0 0 -> xyz=0 0 0.7098668938260085 rpy=0 0 0
- joint Flower_Neighbor: origin xyz=0 1.6505978599657716 0 rpy=0 0 0 -> xyz=0 0 0.8221987201505582 rpy=0 0 0
- joint Fox_Flower: origin xyz=1.4669235270929977 0 0 rpy=0 0 0 -> xyz=0 0 0.8503497477838313 rpy=0 0 0
- joint Impact_Genshin: origin xyz=1.899371955289446 0 0 rpy=0 0 0 -> xyz=0 0 0.706235130180775 rpy=0 0 0
- joint Neighbor_Coffee: origin xyz=0.38963946752698075 0 0 rpy=0 0 0 -> xyz=0 0 0.5263052336564892 rpy=0 0 0
- joint Person_Fox: origin xyz=0 0.12399584576510847 0 rpy=0 0 0 -> xyz=0 0 0.4218871657994694 rpy=0 0 0
- joint Phone_Table: origin xyz=1.9634252835986936 0 0 rpy=0 0 0 -> xyz=0 0 0.7853477184538854 rpy=0 0 0
- joint Table_Impact: origin xyz=0 0.4957528563726159 0 rpy=0 0 0 -> xyz=0 0 0.995775336332686 rpy=0 0 0
- joint Torso_Apple: origin xyz=1.0772888568069745 0 3 rpy=0 0 0 -> xyz=2.609746788032991 0 3 rpy=0 0 0

Commit message: almost done, need to make it random on sides

File: body.urdf (robot description, URDF)
Before this commit: robot robot, 12 links, 11 joints
Links:
- removed link Coffee
- removed link Dog
- removed link Flower
- removed link Fox
- removed link Genshin
- removed link Impact
- removed link Neighbor
- removed link Person
- removed link Phone
- removed link Table
- link Apple: geometry collision box size=1.638818939657638 2.499996005017667 1.6721773065691683; visual box size=1.638818939657638 2.499996005017667 1.6721773065691683
- link Torso: geometry collision box size=0.7119147285502776 1 1; visual box size=0.7119147285502776 1 1
Joints:
- removed joint Apple_Dog
- removed joint Coffee_Phone
- removed joint Dog_Person
- removed joint Flower_Neighbor
- removed joint Fox_Flower
- removed joint Impact_Genshin
- removed joint Neighbor_Coffee
- removed joint Person_Fox
- removed joint Phone_Table
- removed joint Table_Impact
- joint Torso_Apple: origin xyz=2.609746788032991 0 3 rpy=0 0 0 -> xyz=1.3559573642751388 0 3 rpy=0 0 0

Commit message: gonna try something new

File: body.urdf (robot description, URDF)
Before this commit: robot robot, 2 links, 1 joints
Links:
- added link Dog, mass 1; collision box size=0.5297483370694458 0.5676322678561834 0.013921694166750376; visual box size=0.5297483370694458 0.5676322678561834 0.013921694166750376
- added link Flower, mass 1; collision box size=0.5765409739096556 1.5893306213013894 0.21814070723841894; visual box size=0.5765409739096556 1.5893306213013894 0.21814070723841894
- added link Fox, mass 1; collision box size=0.5619307320108782 1.056085198354918 1.423459652167714; visual box size=0.5619307320108782 1.056085198354918 1.423459652167714
- added link Person, mass 1; collision box size=0.3044462066420648 0.03169224140288707 0.9486666046878369; visual box size=0.3044462066420648 0.03169224140288707 0.9486666046878369
- link Apple: geometry collision box size=3.5162553286632057 0.3973093859581889 1.7062548440505134; visual box size=3.5162553286632057 0.3973093859581889 1.7062548440505134
- link Torso: geometry collision box size=1.6345377357969342 1 1; visual box size=1.6345377357969342 1 1
Joints:
- added joint Apple_Dog: type revolute, parent Apple, child Dog, origin xyz=3.5162553286632057 0 0 rpy=0 0 0, axis 0 1 0, limit lower=-3.14159 upper=3.14159 effort=0.0 velocity=0.0
- added joint Dog_Person: type revolute, parent Dog, child Person, origin xyz=0 0 0.013921694166750376 rpy=0 0 0, axis 0 1 0, limit lower=-3.14159 upper=3.14159 effort=0.0 velocity=0.0
- added joint Fox_Flower: type revolute, parent Fox, child Flower, origin xyz=0.2809653660054391 0.528042599177459 0 rpy=0 0 0, axis 0 1 0, limit lower=-3.14159 upper=3.14159 effort=0.0 velocity=0.0
- added joint Person_Fox: type revolute, parent Person, child Fox, origin xyz=0.1522231033210324 0 0.47433330234391846 rpy=0 0 0, axis 0 1 0, limit lower=-3.14159 upper=3.14159 effort=0.0 velocity=0.0
- joint Torso_Apple: origin xyz=1.3559573642751388 0 3 rpy=0 0 0 -> xyz=-1.1827311321015328 0 3 rpy=0 0 0

Commit message: need to fix joints then its done

File: body.urdf (robot description, URDF)
Before this commit: robot robot, 7 links, 6 joints
Links:
- removed link Flower
- removed link Neighbor
- link Apple: geometry collision box size=0.4049230148156777 0.7422121128647636 1.1019353854825014; visual box size=0.4049230148156777 0.7422121128647636 1.1019353854825014
- link Dog: geometry collision box size=1.5409871614434825 0.4401290053663669 0.8959087998005193; visual box size=1.5409871614434825 0.4401290053663669 0.8959087998005193
- link Fox: geometry collision box size=1.8070807464824268 0.38422429587506723 0.6186167241687923; visual box size=1.8070807464824268 0.38422429587506723 0.6186167241687923
- link Person: geometry collision box size=0.42254380065394703 1.0468536195022116 0.25358796256401606; visual box size=0.42254380065394703 1.0468536195022116 0.25358796256401606
- link Torso: geometry collision box size=0.8050706145914097 1 1; visual box size=0.8050706145914097 1 1
Joints:
- removed joint Apple_Dog
- removed joint Dog_Person
- removed joint Flower_Neighbor
- removed joint Fox_Flower
- removed joint Person_Fox
- added joint Apple_Fox: type revolute, parent Apple, child Fox, origin xyz=0.20246150740783886 0.3711060564323818 0 rpy=0 0 0, axis 0 1 0, limit lower=-3.14159 upper=3.14159 effort=0.0 velocity=0.0
- added joint Apple_Person: type revolute, parent Apple, child Person, origin xyz=0.20246150740783886 0 0.5509676927412507 rpy=0 0 0, axis 0 1 0, limit lower=-3.14159 upper=3.14159 effort=0.0 velocity=0.0
- added joint Torso_Dog: type revolute, parent Torso, child Dog, origin xyz=0.40253530729570486 0.5 0 rpy=0 0 0, axis 0 1 0, limit lower=-3.14159 upper=3.14159 effort=0.0 velocity=0.0
- joint Torso_Apple: origin xyz=1.8786579801760201 0 3 rpy=0 0 0 -> xyz=1.4025353072957047 0 3 rpy=0 0 0

Commit message: it breaks when there's more than 2 numoflinks

File: body.urdf (robot description, URDF)
Before this commit: robot robot, 5 links, 4 joints
Links:
- removed link Fox
- removed link Person
- link Apple: geometry collision box size=1.8937541601385064 1.6089569935280186 0.8684920323024694; visual box size=1.8937541601385064 1.6089569935280186 0.8684920323024694
- link Dog: geometry collision box size=1.2281673088087648 1.1819846729307222 1.821574650003046; visual box size=1.2281673088087648 1.1819846729307222 1.821574650003046
- link Torso: geometry collision box size=0.4848608677431725 1 1; visual box size=0.4848608677431725 1 1
Joints:
- removed joint Apple_Fox
- removed joint Apple_Person
- joint Torso_Apple: origin xyz=1.4025353072957047 0 3 rpy=0 0 0 -> xyz=-1.7575695661284136 0 3 rpy=0 0 0
- joint Torso_Dog: origin xyz=0.40253530729570486 0.5 0 rpy=0 0 0 -> xyz=0.5999117109594782 0 0.5 rpy=0 0 0

Commit message: this works sometimes

File: body.urdf (robot description, URDF)
Before this commit: robot robot, 3 links, 2 joints
Links:
- added link Person, mass 1; collision box size=0.8592968238506389 0.7526031113259246 0.5532994518496546; visual box size=0.8592968238506389 0.7526031113259246 0.5532994518496546
- link Apple: geometry collision box size=0.12032724635798764 0.5647345924947773 1.1513510867670431; visual box size=0.12032724635798764 0.5647345924947773 1.1513510867670431
- link Dog: geometry collision box size=0.47060869794135707 0.13742914671373185 1.3174252610046324; visual box size=0.47060869794135707 0.13742914671373185 1.3174252610046324
- link Torso: geometry collision box size=1.7773986272976372 1 1; visual box size=1.7773986272976372 1 1
Joints:
- removed joint Torso_Dog
- added joint Dog_Dog: type revolute, parent Dog, child Dog, origin xyz=0.23530434897067853 0.06871457335686593 0 rpy=0 0 0, axis 0 1 0, limit lower=-3.14159 upper=3.14159 effort=0.0 velocity=0.0
- added joint Torso_Person: type revolute, parent Torso, child Person, origin xyz=0.8886993136488186 0.5 0 rpy=0 0 0, axis 0 1 0, limit lower=-3.14159 upper=3.14159 effort=0.0 velocity=0.0
- joint Torso_Apple: origin xyz=-1.7575695661284136 0 3 rpy=0 0 0 -> xyz=1.8886993136488186 0 3 rpy=0 0 0

Commit message: yes

File: body.urdf (robot description, URDF)
Before this commit: robot robot, 6 links, 5 joints
Links:
- link Apple: geometry collision box size=0.8720542065574857 0.052503366954301356 1.27976416262022; visual box size=0.8720542065574857 0.052503366954301356 1.27976416262022
- link Dog: geometry collision box size=0.8948298573073019 1.7180241536000707 1.285159789490721; visual box size=0.8948298573073019 1.7180241536000707 1.285159789490721
- link Flower: geometry collision box size=0.4199063128666962 0.7574916199114341 0.7007086923229902; visual box size=0.4199063128666962 0.7574916199114341 0.7007086923229902
- link Fox: geometry collision box size=1.724482463195312 0.08917761591992956 1.4469099243747197; visual box size=1.724482463195312 0.08917761591992956 1.4469099243747197
- link Person: geometry collision box size=0.8283901209648761 0.8587700152715694 1.7364198682262222; visual box size=0.8283901209648761 0.8587700152715694 1.7364198682262222
- link Torso: geometry collision box size=0.2029681909370855 1 1; visual box size=0.2029681909370855 1 1
Joints:
- joint Apple_Dog: origin xyz=3.5162553286632057 0 0 rpy=0 0 0 -> xyz=0.8720542065574857 0 0 rpy=0 0 0
- joint Dog_Person: origin xyz=0 0 0.013921694166750376 rpy=0 0 0 -> xyz=0 0 1.285159789490721 rpy=0 0 0
- joint Fox_Flower: origin xyz=0.2809653660054391 0.528042599177459 0 rpy=0 0 0 -> xyz=0.862241231597656 0 0.7234549621873598 rpy=0 0 0
- joint Person_Fox: origin xyz=0.1522231033210324 0 0.47433330234391846 rpy=0 0 0 -> xyz=0 0 1.7364198682262222 rpy=0 0 0
- joint Torso_Apple: origin xyz=-1.1827311321015328 0 3 rpy=0 0 0 -> xyz=3.1014840954685425 0 3 rpy=0 0 0

Commit message: this maybe works

File: body.urdf (robot description, URDF)
Before this commit: robot robot, 7 links, 6 joints
Links:
- removed link Apple
- removed link Neighbor
- link Dog: geometry collision box size=0.04935288093641299 1.0814601650417692 1.2659483474260778; visual box size=0.04935288093641299 1.0814601650417692 1.2659483474260778
- link Flower: geometry collision box size=0.8827870428933999 0.22036105975300746 0.2566763492563495; visual box size=0.8827870428933999 0.22036105975300746 0.2566763492563495
- link Fox: geometry collision box size=1.5489018602343765 1.5447304225571616 0.28983786768430697; visual box size=1.5489018602343765 1.5447304225571616 0.28983786768430697
- link Person: geometry collision box size=0.6409509394652164 0.9443990631049601 1.5314269885406038; visual box size=0.6409509394652164 0.9443990631049601 1.5314269885406038
- link Torso: geometry collision box size=1.1461470143358359 1 1; visual box size=1.1461470143358359 1 1
Joints:
- removed joint Apple_Dog
- removed joint Dog_Person
- removed joint Flower_Neighbor
- removed joint Fox_Flower
- removed joint Person_Fox
- removed joint Torso_Apple
- added joint Dog_Fox: type revolute, parent Dog, child Fox, origin xyz=0.5366020867195914 0.31289573539918614 0.20205043843094606 rpy=0 0 0, axis 0 1 0, limit lower=-3.14159 upper=3.14159 effort=0.0 velocity=0.0
- added joint Fox_Dog: type revolute, parent Fox, child Dog, origin xyz=0.6904901121319319 0.8885085371302035 0.03423222405748849 rpy=0 0 0, axis 0 1 0, limit lower=-3.14159 upper=3.14159 effort=0.0 velocity=0.0
- added joint Fox_Person: type revolute, parent Fox, child Person, origin xyz=0.7744509301171882 0.7723652112785808 0.14491893384215349 rpy=0 0 0, axis 0 1 0, limit lower=-3.14159 upper=3.14159 effort=0.0 velocity=0.0
- added joint Torso_Flower: type revolute, parent Torso, child Flower, origin xyz=0.5730735071679179 0 3 rpy=0 0 0, axis 0 1 0, limit lower=-3.14159 upper=3.14159 effort=0.0 velocity=0.0

Commit message: i think I know what to do

File: body.urdf (robot description, URDF)
Before this commit: robot robot, 6 links, 5 joints
Links:
- added link Coffee, mass 1; collision box size=1.8779407879974348 0.9843438456502118 0.9553256478366638; visual box size=1.8779407879974348 0.9843438456502118 0.9553256478366638
- added link Neighbor, mass 1; collision box size=0.6292328838858745 0.009915401745676178 0.348646885190131; visual box size=0.6292328838858745 0.009915401745676178 0.348646885190131
- added link Phone, mass 1; collision box size=0.856227500589064 0.2587843954868345 0.7179027258265651; visual box size=0.856227500589064 0.2587843954868345 0.7179027258265651
- link Apple: geometry collision box size=1.914898141784688 2.6718498778188335 1.750010630996654; visual box size=1.914898141784688 2.6718498778188335 1.750010630996654
- link Dog: geometry collision box size=0.4562048973075383 0.9355204404417177 1.3751020813599344; visual box size=0.4562048973075383 0.9355204404417177 1.3751020813599344
- link Flower: geometry collision box size=0.6485310563954632 1.1716407006940377 0.7496843999996496; visual box size=0.6485310563954632 1.1716407006940377 0.7496843999996496
- link Fox: geometry collision box size=1.527224808334465 0.09983702094200164 0.313512112684188; visual box size=1.527224808334465 0.09983702094200164 0.313512112684188
- link Person: geometry collision box size=0.5447979667454204 1.0086959102469923 1.1015361439950484; visual box size=0.5447979667454204 1.0086959102469923 1.1015361439950484
- link Torso: geometry collision box size=1.7776246116751764 1 1; visual box size=1.7776246116751764 1 1
Joints:
- added joint Coffee_Phone: type revolute, parent Coffee, child Phone, origin xyz=0 0 0.9553256478366638 rpy=0 0 0, axis 0 1 0, limit lower=-3.14159 upper=3.14159 effort=0.0 velocity=0.0
- added joint Flower_Neighbor: type revolute, parent Flower, child Neighbor, origin xyz=0 0.5858203503470188 0.3748421999998248 rpy=0 0 0, axis 0 1 0, limit lower=-3.14159 upper=3.14159 effort=0.0 velocity=0.0
- added joint Neighbor_Coffee: type revolute, parent Neighbor, child Coffee, origin xyz=0 0.004957700872838089 0.1743234425950655 rpy=0 0 0, axis 0 1 0, limit lower=-3.14159 upper=3.14159 effort=0.0 velocity=0.0
- joint Apple_Dog: origin xyz=3.5162553286632057 0 0 rpy=0 0 0 -> xyz=1.914898141784688 0 0 rpy=0 0 0
- joint Dog_Person: origin xyz=0 0 0.013921694166750376 rpy=0 0 0 -> xyz=0.4562048973075383 0 0 rpy=0 0 0
- joint Fox_Flower: origin xyz=0.2809653660054391 0.528042599177459 0 rpy=0 0 0 -> xyz=0 0 0.313512112684188 rpy=0 0 0
- joint Person_Fox: origin xyz=0.1522231033210324 0 0.47433330234391846 rpy=0 0 0 -> xyz=0.2723989833727102 0 0.5507680719975242 rpy=0 0 0
- joint Torso_Apple: origin xyz=-1.1827311321015328 0 3 rpy=0 0 0 -> xyz=3.8888123058375883 0 3 rpy=0 0 0
