Commit message: this is  done

File: body.urdf (robot description, URDF)
Before this commit: robot robot, 5 links, 4 joints
Links:
- added link Neighbor, mass 1; collision box size=0.4970076209426577 1.1395259463625869 0.49966644930408455; visual box size=0.4970076209426577 1.1395259463625869 0.49966644930408455
- link Dog: geometry collision box size=0.7949930353202577 1.0036984265528823 1.2678187037645505; visual box size=0.7949930353202577 1.0036984265528823 1.2678187037645505
- link Flower: geometry collision box size=1.5535605745862628 0.29377893951351686 0.07836043766925815; visual box size=1.5535605745862628 0.29377893951351686 0.07836043766925815
- link Fox: geometry collision box size=1.1693233668783247 0.0015082346957009385 0.8700333112179344; visual box size=1.1693233668783247 0.0015082346957009385 0.8700333112179344
- link Person: geometry collision box size=0.18453362181191157 1.6211194179313324 1.8214430303726967; visual box size=0.18453362181191157 1.6211194179313324 1.8214430303726967
- link Torso: geometry collision box size=0.1715242756080353 1 1; visual box size=0.1715242756080353 1 1
Joints:
- removed joint Dog_Fox
- removed joint Fox_Dog
- removed joint Fox_Person
- added joint Flower_Dog: type revolute, parent Flower, child Dog, origin xyz=0.7767802872931314 0 0 rpy=0 0 0, axis 0 1 0, limit lower=-3.14159 upper=3.14159 effort=0.0 velocity=0.0
- added joint Neighbor_Person: type revolute, parent Neighbor, child Person, origin xyz=0 0.5697629731812934 0 rpy=0 0 0, axis 0 1 0, limit lower=-3.14159 upper=3.14159 effort=0.0 velocity=0.0
- added joint Torso_Fox: type revolute, parent Torso, child Fox, origin xyz=0 0 0.5 rpy=0 0 0, axis 0 1 0, limit lower=-3.14159 upper=3.14159 effort=0.0 velocity=0.0
- added joint Torso_Neighbor: type revolute, parent Torso, child Neighbor, origin xyz=0.08576213780401765 0 3 rpy=0 0 0, axis 0 1 0, limit lower=-3.14159 upper=3.14159 effort=0.0 velocity=0.0
- joint Torso_Flower: origin xyz=0.5730735071679179 0 3 rpy=0 0 0 -> xyz=0 0.5 0 rpy=0 0 0

Commit message: meow

File: body.urdf (robot description, URDF)
Before this commit: robot robot, 9 links, 8 joints
Links:
- removed link Coffee
- removed link Neighbor
- removed link Phone
- link Apple: geometry collision box size=0.5726375868065503 3.2453103831558328 2.291157374883737; visual box size=0.5726375868065503 3.2453103831558328 2.291157374883737
- link Dog: geometry collision box size=0.9665164315475634 0.8953434476834967 1.5581533480740033; visual box size=0.9665164315475634 0.8953434476834967 1.5581533480740033
- link Flower: geometry collision box size=0.8504287695120043 0.018102732577588432 0.4393785790318985; visual box size=0.8504287695120043 0.018102732577588432 0.4393785790318985
- link Fox: geometry collision box size=0.5064072585945107 0.9281959503145367 1.4543463526079956; visual box size=0.5064072585945107 0.9281959503145367 1.4543463526079956
- link Person: geometry collision box size=1.196671115526762 1.3738867190881363 0.887118086967603; visual box size=1.196671115526762 1.3738867190881363 0.887118086967603
- link Torso: geometry collision box size=0.8621529399251151 1 1; visual box size=0.8621529399251151 1 1
Joints:
- removed joint Coffee_Phone
- removed joint Flower_Neighbor
- removed joint Neighbor_Coffee
- joint Apple_Dog: origin xyz=1.914898141784688 0 0 rpy=0 0 0 -> xyz=0.5726375868065503 0 0 rpy=0 0 0
- joint Dog_Person: origin xyz=0.4562048973075383 0 0 rpy=0 0 0 -> xyz=0 0 1.5581533480740033 rpy=0 0 0
- joint Fox_Flower: origin xyz=0 0 0.313512112684188 rpy=0 0 0 -> xyz=0.5064072585945107 0 0 rpy=0 0 0
- joint Person_Fox: origin xyz=0.2723989833727102 0 0.5507680719975242 rpy=0 0 0 -> xyz=0.598335557763381 0 0.4435590434838015 rpy=0 0 0
- joint Torso_Apple: origin xyz=3.8888123058375883 0 3 rpy=0 0 0 -> xyz=-3.5689235300374422 0 3 rpy=0 0 0

Commit message: yes

File: body.urdf (robot description, URDF)
Before this commit: robot robot, 6 links, 5 joints
Links:
- removed link Flower
- removed link Fox
- removed link Neighbor
- removed link Person
- link Dog: geometry collision box size=1.2110871758006876 0.06591849723060594 1.0178349852779334; visual box size=1.2110871758006876 0.06591849723060594 1.0178349852779334
- link Torso: geometry collision box size=1.4982470538409607 1 1; visual box size=1.4982470538409607 1 1
Joints:
- removed joint Flower_Dog
- removed joint Neighbor_Person
- removed joint Torso_Flower
- removed joint Torso_Fox
- removed joint Torso_Neighbor
- added joint Torso_Dog: type revolute, parent Torso, child Dog, origin xyz=1.7491235269204803 0 3 rpy=0 0 0, axis 0 1 0, limit lower=-3.14159 upper=3.14159 effort=0.0 velocity=0.0

Commit message: yes

File: body.urdf (robot description, URDF)
Before this commit: robot robot, 9 links, 8 joints
Links:
- removed link Coffee
- removed link Flower
- removed link Fox
- removed link Neighbor
- removed link Person
- removed link Phone
- link Apple: geometry collision box size=0.2337016380563659 1.8859439852120157 3.3321346832457555; visual box size=0.2337016380563659 1.8859439852120157 3.3321346832457555
- link Dog: geometry collision box size=1.383311530310603 0.08750162721662003 1.8948766934368992; visual box size=1.383311530310603 0.08750162721662003 1.8948766934368992
- link Torso: geometry collision box size=1.2925999732230056 1 1; visual box size=1.2925999732230056 1 1
Joints:
- removed joint Coffee_Phone
- removed joint Dog_Person
- removed joint Flower_Neighbor
- removed joint Fox_Flower
- removed joint Neighbor_Coffee
- removed joint Person_Fox
- joint Apple_Dog: origin xyz=1.914898141784688 0 0 rpy=0 0 0 -> xyz=0.2337016380563659 0 0 rpy=0 0 0
- joint Torso_Apple: origin xyz=3.8888123058375883 0 3 rpy=0 0 0 -> xyz=3.6462999866115027 0 3 rpy=0 0 0

Commit message: yes

File: body.urdf (robot description, URDF)
Before this commit: robot robot, 2 links, 1 joints
Links:
- link Dog: geometry collision box size=0.2664337223152242 1.6809028294414214 1.274799642627927; visual box size=0.2664337223152242 1.6809028294414214 1.274799642627927
- link Torso: geometry collision box size=0.6612368025007893 1 1; visual box size=0.6612368025007893 1 1
Joints:
- joint Torso_Dog: origin xyz=1.7491235269204803 0 3 rpy=0 0 0 -> xyz=0 0.5 0 rpy=0 0 0

Commit message: just added some minor changes

File: body.urdf (robot description, URDF)
Before this commit: robot robot, 3 links, 2 joints
Links:
- added link Flower, mass 1; collision box size=1.9834318828066608 0.4439440303617985 0.22296812750284034; visual box size=1.9834318828066608 0.4439440303617985 0.22296812750284034
- added link Fox, mass 1; collision box size=1.3473003176762264 1.7151071102460107 0.11934968269774049; visual box size=1.3473003176762264 1.7151071102460107 0.11934968269774049
- added link Person, mass 1; collision box size=1.9876922545454383 0.9206331262116518 1.8896638848274647; visual box size=1.9876922545454383 0.9206331262116518 1.8896638848274647
- link Apple: geometry collision box size=3.082728671947827 0.6357601522902936 2.7206027226044216; visual box size=3.082728671947827 0.6357601522902936 2.7206027226044216
- link Dog: geometry collision box size=0.32892764755244697 0.39764285724285275 1.7735391653502035; visual box size=0.32892764755244697 0.39764285724285275 1.7735391653502035
- link Torso: geometry collision box size=1.2825508357682418 1 1; visual box size=1.2825508357682418 1 1
Joints:
- added joint Dog_Person: type revolute, parent Dog, child Person, origin xyz=0.16446382377622348 0 0.8867695826751018 rpy=0 0 0, axis 0 1 0, limit lower=-3.14159 upper=3.14159 effort=0.0 velocity=0.0
- added joint Fox_Flower: type revolute, parent Fox, child Flower, origin xyz=0 0 0.11934968269774049 rpy=0 0 0, axis 0 1 0, limit lower=-3.14159 upper=3.14159 effort=0.0 velocity=0.0
- added joint Person_Fox: type revolute, parent Person, child Fox, origin xyz=0.9938461272727191 0 0.9448319424137324 rpy=0 0 0, axis 0 1 0, limit lower=-3.14159 upper=3.14159 effort=0.0 velocity=0.0
- joint Apple_Dog: origin xyz=0.2337016380563659 0 0 rpy=0 0 0 -> xyz=3.082728671947827 0 0 rpy=0 0 0
- joint Torso_Apple: origin xyz=3.6462999866115027 0 3 rpy=0 0 0 -> xyz=-0.3587245821158791 0 3 rpy=0 0 0

Commit message: added some print statements, gonna start working on the mutate function now

File: body.urdf (robot description, URDF)
Before this commit: robot robot, 6 links, 5 joints
Links:
- link Apple: geometry collision box size=1.4917672837190041 0.8622480066357454 1.888486520931211; visual box size=1.4917672837190041 0.8622480066357454 1.888486520931211
- link Dog: geometry collision box size=0.23903500371561504 1.739914454833909 1.3021198794917666; visual box size=0.23903500371561504 1.739914454833909 1.3021198794917666
- link Flower: geometry collision box size=1.155168324261267 1.2108322685477246 0.7856453112113286; visual box size=1.155168324261267 1.2108322685477246 0.7856453112113286
- link Fox: geometry collision box size=0.6995474320391053 0.14450273031712668 1.0825175325178407; visual box size=0.6995474320391053 0.14450273031712668 1.0825175325178407
- link Person: geometry collision box size=0.8553289984331005 0.7087980295364331 0.3540011247308066; visual box size=0.8553289984331005 0.7087980295364331 0.3540011247308066
- link Torso: geometry collision box size=1.1300249836352476 1 1; visual box size=1.1300249836352476 1 1
Joints:
- joint Apple_Dog: origin xyz=3.082728671947827 0 0 rpy=0 0 0 -> xyz=1.4917672837190041 0 0 rpy=0 0 0
- joint Dog_Person: origin xyz=0.16446382377622348 0 0.8867695826751018 rpy=0 0 0 -> xyz=0 1.739914454833909 0 rpy=0 0 0
- joint Fox_Flower: origin xyz=0 0 0.11934968269774049 rpy=0 0 0 -> xyz=0 0.14450273031712668 0 rpy=0 0 0
- joint Person_Fox: origin xyz=0.9938461272727191 0 0.9448319424137324 rpy=0 0 0 -> xyz=0 0.7087980295364331 0 rpy=0 0 0
- joint Torso_Apple: origin xyz=-0.3587245821158791 0 3 rpy=0 0 0 -> xyz=2.565012491817624 0 3 rpy=0 0 0

Commit message: gonna try something new

File: body.urdf (robot description, URDF)
Before this commit: robot robot, 6 links, 5 joints
Links:
- added link Grace, mass 1; collision box size=3.686599197740934 2.9711778124320127 0.6157504892310453; visual box size=3.686599197740934 2.9711778124320127 0.6157504892310453
- link Apple: geometry collision box size=1.4289226480392307 3.198712692001551 0.921021439981033; visual box size=1.4289226480392307 3.198712692001551 0.921021439981033
- link Dog: geometry collision box size=1.3268553584637672 1.8431532170011118 0.09183532934833338; visual box size=1.3268553584637672 1.8431532170011118 0.09183532934833338
- link Flower: geometry collision box size=1.0447683328548014 1.7178748599198914 0.43626327646304786; visual box size=1.0447683328548014 1.7178748599198914 0.43626327646304786
- link Fox: geometry collision box size=1.0239592967983149 0.9828143634521744 0.3302669714954074; visual box size=1.0239592967983149 0.9828143634521744 0.3302669714954074
- link Person: geometry collision box size=1.978569298835041 1.9193812429036747 0.10519149807181827; visual box size=1.978569298835041 1.9193812429036747 0.10519149807181827
- link Torso: geometry collision box size=1.841199786201208 1 1; visual box size=1.841199786201208 1 1
Joints:
- added joint Person_Grace: type revolute, parent Person, child Grace, origin xyz=0.9892846494175205 0.9596906214518374 0 rpy=0 0 0, axis 0 1 0, limit lower=-3.14159 upper=3.14159 effort=0.0 velocity=0.0
- joint Apple_Dog: origin xyz=1.4917672837190041 0 0 rpy=0 0 0 -> xyz=1.4289226480392307 0 0 rpy=0 0 0
- joint Dog_Person: origin xyz=0 1.739914454833909 0 rpy=0 0 0 -> xyz=1.3268553584637672 0 0 rpy=0 0 0
- joint Fox_Flower: origin xyz=0 0.14450273031712668 0 rpy=0 0 0 -> xyz=0 0.4914071817260872 0.1651334857477037 rpy=0 0 0
- joint Person_Fox: origin xyz=0 0.7087980295364331 0 rpy=0 0 0 -> xyz=0.9892846494175205 0 0.052595749035909134 rpy=0 0 0
- joint Torso_Apple: origin xyz=2.565012491817624 0 3 rpy=0 0 0 -> xyz=-3.079400106899396 0 3 rpy=0 0 0

Commit message: need to fix the file readings

File: body.urdf (robot description, URDF)
Before this commit: robot robot, 7 links, 6 joints
Links:
- removed link Grace
- link Apple: geometry collision box size=1.7419522710718818 0.6619953586247904 3.286296338418801; visual box size=1.7419522710718818 0.6619953586247904 3.286296338418801
- link Dog: geometry collision box size=1.1218060328204456 1.978220924842337 0.2558528080402629; visual box size=1.1218060328204456 1.978220924842337 0.2558528080402629
- link Flower: geometry collision box size=1.7891607773854201 0.205913914700103 1.3867468373971825; visual box size=1.7891607773854201 0.205913914700103 1.3867468373971825
- link Fox: geometry collision box size=1.7984717579979057 0.413368235983433 0.08400585286572038; visual box size=1.7984717579979057 0.413368235983433 0.08400585286572038
- link Person: geometry collision box size=1.4102749396501604 1.9041334693049015 1.7819504202812844; visual box size=1.4102749396501604 1.9041334693049015 1.7819504202812844
- link Torso: geometry collision box size=1.3541165158898618 1 1; visual box size=1.3541165158898618 1 1
Joints:
- removed joint Person_Grace
- joint Apple_Dog: origin xyz=1.4289226480392307 0 0 rpy=0 0 0 -> xyz=1.7419522710718818 0 0 rpy=0 0 0
- joint Dog_Person: origin xyz=1.3268553584637672 0 0 rpy=0 0 0 -> xyz=0.5609030164102228 0.9891104624211685 0 rpy=0 0 0
- joint Fox_Flower: origin xyz=0 0.4914071817260872 0.1651334857477037 rpy=0 0 0 -> xyz=0 0.2066841179917165 0.04200292643286019 rpy=0 0 0
- joint Person_Fox: origin xyz=0.9892846494175205 0 0.052595749035909134 rpy=0 0 0 -> xyz=0.7051374698250802 0 0.8909752101406422 rpy=0 0 0
- joint Torso_Apple: origin xyz=-3.079400106899396 0 3 rpy=0 0 0 -> xyz=0.6770582579449309 0 3 rpy=0 0 0

Commit message: yeah this didnt' work

File: body.urdf (robot description, URDF)
Before this commit: robot robot, 6 links, 5 joints
Links:
- link Apple: geometry collision box size=0.8461464471317499 0.06737992254113401 0.33548811352748986; visual box size=0.8461464471317499 0.06737992254113401 0.33548811352748986
- link Dog: geometry collision box size=1.824908212963387 0.6518610597362913 0.9815358467336979; visual box size=1.824908212963387 0.6518610597362913 0.9815358467336979
- link Flower: geometry collision box size=1.2560359261683982 1.848024913092329 1.6429834414990052; visual box size=1.2560359261683982 1.848024913092329 1.6429834414990052
- link Fox: geometry collision box size=1.4532903014749559 0.12873188782964262 0.8701630820184716; visual box size=1.4532903014749559 0.12873188782964262 0.8701630820184716
- link Person: geometry collision box size=0.2763260933421958 1.97929777597884 0.33425400129039384; visual box size=0.2763260933421958 1.97929777597884 0.33425400129039384
- link Torso: geometry collision box size=1.9554698267430963 1 1; visual box size=1.9554698267430963 1 1
Joints:
- joint Apple_Dog: origin xyz=1.7419522710718818 0 0 rpy=0 0 0 -> xyz=0.8461464471317499 0 0 rpy=0 0 0
- joint Dog_Person: origin xyz=0.5609030164102228 0.9891104624211685 0 rpy=0 0 0 -> xyz=0 0 0.9815358467336979 rpy=0 0 0
- joint Fox_Flower: origin xyz=0 0.2066841179917165 0.04200292643286019 rpy=0 0 0 -> xyz=0.7266451507374779 0.06436594391482131 0 rpy=0 0 0
- joint Person_Fox: origin xyz=0.7051374698250802 0 0.8909752101406422 rpy=0 0 0 -> xyz=0 0.98964888798942 0.16712700064519692 rpy=0 0 0
- joint Torso_Apple: origin xyz=0.6770582579449309 0 3 rpy=0 0 0 -> xyz=0.9777349133715482 0 3 rpy=0 0 0

Commit message: was able to store everything, time to start modifying the body parts

File: body.urdf (robot description, URDF)
Before this commit: robot robot, 7 links, 6 joints
Links:
- removed link Grace
- link Apple: geometry collision box size=0.7570072449020175 2.1645979735330445 0.9475704652643557; visual box size=0.7570072449020175 2.1645979735330445 0.9475704652643557
- link Dog: geometry collision box size=0.3811240542131684 1.7822142988870833 1.3888554778186772; visual box size=0.3811240542131684 1.7822142988870833 1.3888554778186772
- link Flower: geometry collision box size=1.1805912722223688 1.1901065032962639 0.22579392704037415; visual box size=1.1805912722223688 1.1901065032962639 0.22579392704037415
- link Fox: geometry collision box size=0.7974139787727599 1.9643076925794898 0.04758326204301455; visual box size=0.7974139787727599 1.9643076925794898 0.04758326204301455
- link Person: geometry collision box size=1.6948914101650239 0.819455249809768 1.50962894077908; visual box size=1.6948914101650239 0.819455249809768 1.50962894077908
- link Torso: geometry collision box size=1.9303505685873374 1 1; visual box size=1.9303505685873374 1 1
Joints:
- removed joint Person_Grace
- joint Apple_Dog: origin xyz=1.4289226480392307 0 0 rpy=0 0 0 -> xyz=0.7570072449020175 0 0 rpy=0 0 0
- joint Dog_Person: origin xyz=1.3268553584637672 0 0 rpy=0 0 0 -> xyz=0.1905620271065842 0 0.6944277389093386 rpy=0 0 0
- joint Fox_Flower: origin xyz=0 0.4914071817260872 0.1651334857477037 rpy=0 0 0 -> xyz=0.39870698938637994 0 0.023791631021507276 rpy=0 0 0
- joint Person_Fox: origin xyz=0.9892846494175205 0 0.052595749035909134 rpy=0 0 0 -> xyz=0 0 1.50962894077908 rpy=0 0 0
- joint Torso_Apple: origin xyz=-3.079400106899396 0 3 rpy=0 0 0 -> xyz=-3.034824715706331 0 3 rpy=0 0 0

Commit message: finished saving everything into arrays, time to delete the calls to cubes and joints and make them in a for loop

File: body.urdf (robot description, URDF)
Before this commit: robot robot, 6 links, 5 joints
Links:
- added link Grace, mass 1; collision box size=1.1691682770525715 1.5449116020082125 0.34637152629693135; visual box size=1.1691682770525715 1.5449116020082125 0.34637152629693135
- added link Learn, mass 1; collision box size=3.3706728601948948 0.6132537851175615 1.3460873867463894; visual box size=3.3706728601948948 0.6132537851175615 1.3460873867463894
- link Apple: geometry collision box size=1.9426626838774683 1.5552175099624495 2.28720319411345; visual box size=1.9426626838774683 1.5552175099624495 2.28720319411345
- link Dog: geometry collision box size=0.7092266612151337 0.9020553714686206 0.7508814131460351; visual box size=0.7092266612151337 0.9020553714686206 0.7508814131460351
- link Flower: geometry collision box size=1.2020179864670373 0.694732845117038 1.9564876564563272; visual box size=1.2020179864670373 0.694732845117038 1.9564876564563272
- link Fox: geometry collision box size=1.4262495111734514 0.7938241601649014 0.6962327957095391; visual box size=1.4262495111734514 0.7938241601649014 0.6962327957095391
- link Person: geometry collision box size=0.8334221775370363 1.9409106057282621 1.253103129023546; visual box size=0.8334221775370363 1.9409106057282621 1.253103129023546
- link Torso: geometry collision box size=0.4360771402363559 1 1; visual box size=0.4360771402363559 1 1
Joints:
- added joint Fox_Yoojin: type revolute, parent Fox, child Yoojin, origin xyz=0 0.3969120800824507 0.34811639785476955 rpy=0 0 0, axis 0 1 0, limit lower=-3.14159 upper=3.14159 effort=0.0 velocity=0.0
- added joint Person_Grace: type revolute, parent Person, child Grace, origin xyz=0.41671108876851815 0.9704553028641311 0 rpy=0 0 0, axis 0 1 0, limit lower=-3.14159 upper=3.14159 effort=0.0 velocity=0.0
- joint Apple_Dog: origin xyz=0.7570072449020175 0 0 rpy=0 0 0 -> xyz=1.9426626838774683 0 0 rpy=0 0 0
- joint Dog_Person: origin xyz=0.1905620271065842 0 0.6944277389093386 rpy=0 0 0 -> xyz=0.7092266612151337 0 0 rpy=0 0 0
- joint Fox_Flower: origin xyz=0.39870698938637994 0 0.023791631021507276 rpy=0 0 0 -> xyz=0 0.3969120800824507 0.34811639785476955 rpy=0 0 0
- joint Person_Fox: origin xyz=0 0 1.50962894077908 rpy=0 0 0 -> xyz=0.41671108876851815 0.9704553028641311 0 rpy=0 0 0
- joint Torso_Apple: origin xyz=-3.034824715706331 0 3 rpy=0 0 0 -> xyz=-0.781961429881822 0 3 rpy=0 0 0

Commit message: something wrong with the body.urdf

File: body.urdf (robot description, URDF)
Before this commit: robot robot, 8 links, 7 joints
Links:
- removed link Learn
- link Apple: geometry collision box size=2.6541573944487213 0.10258829597417707 2.933447088997999; visual box size=2.6541573944487213 0.10258829597417707 2.933447088997999
- link Dog: geometry collision box size=0.6382803577244307 0.23023925753222962 1.2558082182179529; visual box size=0.6382803577244307 0.23023925753222962 1.2558082182179529
- link Flower: geometry collision box size=0.10963485133144024 1.355138438304882 0.8464511629636702; visual box size=0.10963485133144024 1.355138438304882 0.8464511629636702
- link Fox: geometry collision box size=1.69127881767463 1.913420624405467 0.29922344273808554; visual box size=1.69127881767463 1.913420624405467 0.29922344273808554
- link Grace: geometry collision box size=1.550422742417267 2.592390530836017 0.17818871607612818; visual box size=1.550422742417267 2.592390530836017 0.17818871607612818
- link Person: geometry collision box size=1.608835072914251 0.41437147797044704 0.9980820620127429; visual box size=1.608835072914251 0.41437147797044704 0.9980820620127429
- link Torso: geometry collision box size=0.3677554211253753 1 1; visual box size=0.3677554211253753 1 1
Joints:
- removed joint Fox_Yoojin
- joint Apple_Dog: origin xyz=1.9426626838774683 0 0 rpy=0 0 0 -> xyz=2.6541573944487213 0 0 rpy=0 0 0
- joint Dog_Person: origin xyz=0.7092266612151337 0 0 rpy=0 0 0 -> xyz=0.31914017886221535 0 0.6279041091089764 rpy=0 0 0
- joint Fox_Flower: origin xyz=0 0.3969120800824507 0.34811639785476955 rpy=0 0 0 -> xyz=0 0 0.29922344273808554 rpy=0 0 0
- joint Person_Fox: origin xyz=0.41671108876851815 0.9704553028641311 0 rpy=0 0 0 -> xyz=0.8044175364571255 0 0.4990410310063714 rpy=0 0 0
- joint Person_Grace: origin xyz=0.41671108876851815 0.9704553028641311 0 rpy=0 0 0 -> xyz=0.1936424244019883 0.4677500998809513 0 rpy=0 0 0
- joint Torso_Apple: origin xyz=-0.781961429881822 0 3 rpy=0 0 0 -> xyz=1.1838777105626876 0 3 rpy=0 0 0
