Commit message: blah

File: body.urdf (robot description, URDF)
Before this commit: robot robot, 7 links, 6 joints
Links:
- link Apple: geometry collision box size=0.722018225832644 1.7829732646289091 2.878208665105674; visual box size=0.722018225832644 1.7829732646289091 2.878208665105674
- link Dog: geometry collision box size=0.31007905239997613 1.2383290589562221 0.3757641076287517; visual box size=0.31007905239997613 1.2383290589562221 0.3757641076287517
- link Flower: geometry collision box size=1.3149390381086583 0.5272194375489725 0.3303081246035806; visual box size=1.3149390381086583 0.5272194375489725 0.3303081246035806
- link Fox: geometry collision box size=0.4284210947586342 0.331414917567066 0.44637109024140353; visual box size=0.4284210947586342 0.331414917567066 0.44637109024140353
- link Grace: geometry collision box size=2.907480042849991 3.7737478597971497 1.4526807250984959; visual box size=2.907480042849991 3.7737478597971497 1.4526807250984959
- link Person: geometry collision box size=0.34220790722942973 1.5368215978602018 0.9934355641571544; visual box size=0.34220790722942973 1.5368215978602018 0.9934355641571544
- link Torso: geometry collision box size=0.029567070631553394 1 1; visual box size=0.029567070631553394 1 1
Joints:
- joint Apple_Dog: origin xyz=1.4289226480392307 0 0 rpy=0 0 0 -> xyz=0.722018225832644 0 0 rpy=0 0 0
- joint Dog_Person: origin xyz=1.3268553584637672 0 0 rpy=0 0 0 -> xyz=0.31007905239997613 0 0 rpy=0 0 0
- joint Fox_Flower: origin xyz=0 0.4914071817260872 0.1651334857477037 rpy=0 0 0 -> xyz=0.2142105473793171 0 0.22318554512070177 rpy=0 0 0
- joint Person_Fox: origin xyz=0.9892846494175205 0 0.052595749035909134 rpy=0 0 0 -> xyz=0.17110395361471487 0 0.4967177820785772 rpy=0 0 0
- joint Person_Grace: origin xyz=0.9892846494175205 0.9596906214518374 0 rpy=0 0 0 -> xyz=0.17110395361471487 0.7684107989301009 0 rpy=0 0 0
- joint Torso_Apple: origin xyz=-3.079400106899396 0 3 rpy=0 0 0 -> xyz=3.0147835353157766 0 3 rpy=0 0 0

Commit message: keeps appending to the end of the body.urdf '

File: body.urdf (robot description, URDF)
Before this commit: robot robot, 7 links, 6 joints
Links:
- removed link Grace
- link Apple: geometry collision box size=0.04400633577799162 3.6119775878734726 2.1273516480942516; visual box size=0.04400633577799162 3.6119775878734726 2.1273516480942516
- link Dog: geometry collision box size=1.5418911447827548 1.1655049872352985 1.3901353457315315; visual box size=1.5418911447827548 1.1655049872352985 1.3901353457315315
- link Flower: geometry collision box size=1.072244293139803 1.5541574925240609 0.44195405280035893; visual box size=1.072244293139803 1.5541574925240609 0.44195405280035893
- link Fox: geometry collision box size=0.31178362853438046 0.39862059685649753 0.6919378842108539; visual box size=0.31178362853438046 0.39862059685649753 0.6919378842108539
- link Person: geometry collision box size=0.8571247263221387 0.29767815532143427 0.3579698069705588; visual box size=0.8571247263221387 0.29767815532143427 0.3579698069705588
- link Torso: geometry collision box size=0.25776646282999116 1 1; visual box size=0.25776646282999116 1 1
Joints:
- removed joint Person_Grace
- joint Apple_Dog: origin xyz=2.6541573944487213 0 0 rpy=0 0 0 -> xyz=0.04400633577799162 0 0 rpy=0 0 0
- joint Dog_Person: origin xyz=0.31914017886221535 0 0.6279041091089764 rpy=0 0 0 -> xyz=0 0 1.3901353457315315 rpy=0 0 0
- joint Fox_Flower: origin xyz=0 0 0.29922344273808554 rpy=0 0 0 -> xyz=0.15589181426719023 0 0.34596894210542695 rpy=0 0 0
- joint Person_Fox: origin xyz=0.8044175364571255 0 0.4990410310063714 rpy=0 0 0 -> xyz=0.4285623631610693 0 0.1789849034852794 rpy=0 0 0
- joint Torso_Apple: origin xyz=1.1838777105626876 0 3 rpy=0 0 0 -> xyz=0.12888323141499558 0 3 rpy=0 0 0

Commit message: blargh

File: body.urdf (robot description, URDF)
Before this commit: robot robot, 7 links, 6 joints
Links:
- link Apple: geometry collision box size=0.25949671180094747 0.7995958500660318 0.34153807524051727; visual box size=0.25949671180094747 0.7995958500660318 0.34153807524051727
- link Dog: geometry collision box size=0.8963716648437006 1.2569138226690917 1.1943786670216834; visual box size=0.8963716648437006 1.2569138226690917 1.1943786670216834
- link Flower: geometry collision box size=0.18033306010120254 1.4346080964160957 1.9260117306454307; visual box size=0.18033306010120254 1.4346080964160957 1.9260117306454307
- link Fox: geometry collision box size=0.7433052094741137 1.0700024345732875 0.9819744794551764; visual box size=0.7433052094741137 1.0700024345732875 0.9819744794551764
- link Grace: geometry collision box size=1.2932915007359154 2.4828897571469026 1.170070396731627; visual box size=1.2932915007359154 2.4828897571469026 1.170070396731627
- link Person: geometry collision box size=1.4796333569069997 0.8578274783886124 0.01475127752002603; visual box size=1.4796333569069997 0.8578274783886124 0.01475127752002603
- link Torso: geometry collision box size=1.8729819235872311 1 1; visual box size=1.8729819235872311 1 1
Joints:
- joint Apple_Dog: origin xyz=0.722018225832644 0 0 rpy=0 0 0 -> xyz=0.25949671180094747 0 0 rpy=0 0 0
- joint Dog_Person: origin xyz=0.31007905239997613 0 0 rpy=0 0 0 -> xyz=0.8963716648437006 0 0 rpy=0 0 0
- joint Fox_Flower: origin xyz=0.2142105473793171 0 0.22318554512070177 rpy=0 0 0 -> xyz=0 0 0.9819744794551764 rpy=0 0 0
- joint Person_Fox: origin xyz=0.17110395361471487 0 0.4967177820785772 rpy=0 0 0 -> xyz=0.7398166784534999 0 0.007375638760013015 rpy=0 0 0
- joint Person_Grace: origin xyz=0.17110395361471487 0.7684107989301009 0 rpy=0 0 0 -> xyz=0.7398166784534999 0.4289137391943062 0 rpy=0 0 0
- joint Torso_Apple: origin xyz=3.0147835353157766 0 3 rpy=0 0 0 -> xyz=-0.06350903820638443 0 3 rpy=0 0 0

Commit message: idk why that fixed the issue but cool

File: body.urdf (robot description, URDF)
Before this commit: robot robot, 6 links, 5 joints
Links:
- link Apple: geometry collision box size=3.9785285584626706 2.209864097117374 1.4894639482589822; visual box size=3.9785285584626706 2.209864097117374 1.4894639482589822
- link Dog: geometry collision box size=0.4610682917697435 0.37302711957416324 1.855159965057633; visual box size=0.4610682917697435 0.37302711957416324 1.855159965057633
- link Flower: geometry collision box size=0.036604389422004946 1.4443292299170438 0.4976798713937287; visual box size=0.036604389422004946 1.4443292299170438 0.4976798713937287
- link Fox: geometry collision box size=0.3554859135086357 0.3845485054779194 0.8514838132519895; visual box size=0.3554859135086357 0.3845485054779194 0.8514838132519895
- link Person: geometry collision box size=1.1236949157925635 0.737887240297388 0.17997182372260534; visual box size=1.1236949157925635 0.737887240297388 0.17997182372260534
- link Torso: geometry collision box size=1.6221957350400107 1 1; visual box size=1.6221957350400107 1 1
Joints:
- joint Apple_Dog: origin xyz=0.04400633577799162 0 0 rpy=0 0 0 -> xyz=3.9785285584626706 0 0 rpy=0 0 0
- joint Dog_Person: origin xyz=0 0 1.3901353457315315 rpy=0 0 0 -> xyz=0 0 1.855159965057633 rpy=0 0 0
- joint Fox_Flower: origin xyz=0.15589181426719023 0 0.34596894210542695 rpy=0 0 0 -> xyz=0.17774295675431784 0 0.42574190662599476 rpy=0 0 0
- joint Person_Fox: origin xyz=0.4285623631610693 0 0.1789849034852794 rpy=0 0 0 -> xyz=0 0 0.17997182372260534 rpy=0 0 0
- joint Torso_Apple: origin xyz=0.12888323141499558 0 3 rpy=0 0 0 -> xyz=-1.1889021324799947 0 3 rpy=0 0 0

Commit message: meow

File: body.urdf (robot description, URDF)
Before this commit: robot robot, 6 links, 5 joints
Links:
- link Apple: geometry collision box size=3.6573237918235595 1.814903255777974 2.4371667269586816; visual box size=3.6573237918235595 1.814903255777974 2.4371667269586816
- link Dog: geometry collision box size=1.1270740041528884 1.6296543165479835 1.1442990659200023; visual box size=1.1270740041528884 1.6296543165479835 1.1442990659200023
- link Flower: geometry collision box size=1.8660218542196039 0.7228889017448317 1.5484863734632262; visual box size=1.8660218542196039 0.7228889017448317 1.5484863734632262
- link Fox: geometry collision box size=1.9467242185168563 1.7535579890328692 0.8647957507309558; visual box size=1.9467242185168563 1.7535579890328692 0.8647957507309558
- link Person: geometry collision box size=1.3344046136673766 1.2828033794837475 1.8516570473190574; visual box size=1.3344046136673766 1.2828033794837475 1.8516570473190574
- link Torso: geometry collision box size=0.8407575214221144 1 1; visual box size=0.8407575214221144 1 1
Joints:
- joint Apple_Dog: origin xyz=3.9785285584626706 0 0 rpy=0 0 0 -> xyz=3.6573237918235595 0 0 rpy=0 0 0
- joint Dog_Person: origin xyz=0 0 1.855159965057633 rpy=0 0 0 -> xyz=0.5635370020764442 0.8148271582739918 0 rpy=0 0 0
- joint Fox_Flower: origin xyz=0.17774295675431784 0 0.42574190662599476 rpy=0 0 0 -> xyz=0 0 0.8647957507309558 rpy=0 0 0
- joint Person_Fox: origin xyz=0 0 0.17997182372260534 rpy=0 0 0 -> xyz=0.6672023068336883 0 0.9258285236595287 rpy=0 0 0
- joint Torso_Apple: origin xyz=-1.1889021324799947 0 3 rpy=0 0 0 -> xyz=0.4203787607110572 0 3 rpy=0 0 0

Commit message: okay I think I know what is going wrong

File: body.urdf (robot description, URDF)
Before this commit: robot robot, 7 links, 6 joints
Links:
- removed link Grace
- link Apple: geometry collision box size=2.3060009421767065 2.2383312333699656 1.8539977621906996; visual box size=2.3060009421767065 2.2383312333699656 1.8539977621906996
- link Dog: geometry collision box size=0.7925075418078824 0.1853823349712267 1.0711189598898159; visual box size=0.7925075418078824 0.1853823349712267 1.0711189598898159
- link Flower: geometry collision box size=0.5286656003674075 0.4589293904394738 0.6139702658028487; visual box size=0.5286656003674075 0.4589293904394738 0.6139702658028487
- link Fox: geometry collision box size=1.218382431104458 0.9194716250866066 0.4120231075282814; visual box size=1.218382431104458 0.9194716250866066 0.4120231075282814
- link Person: geometry collision box size=0.010797998458632385 1.1570746784099473 1.0745377276374548; visual box size=0.010797998458632385 1.1570746784099473 1.0745377276374548
- link Torso: geometry collision box size=0.30745378849755634 1 1; visual box size=0.30745378849755634 1 1
Joints:
- removed joint Person_Grace
- joint Apple_Dog: origin xyz=0.25949671180094747 0 0 rpy=0 0 0 -> xyz=2.3060009421767065 0 0 rpy=0 0 0
- joint Dog_Person: origin xyz=0.8963716648437006 0 0 rpy=0 0 0 -> xyz=0.3962537709039412 0.09269116748561335 0 rpy=0 0 0
- joint Fox_Flower: origin xyz=0 0 0.9819744794551764 rpy=0 0 0 -> xyz=0 0 0.4120231075282814 rpy=0 0 0
- joint Person_Fox: origin xyz=0.7398166784534999 0 0.007375638760013015 rpy=0 0 0 -> xyz=0.005398999229316193 0 0.5372688638187274 rpy=0 0 0
- joint Torso_Apple: origin xyz=-0.06350903820638443 0 3 rpy=0 0 0 -> xyz=3.153726894248778 0 3 rpy=0 0 0

Commit message: i hate that the error was this dumb

File: body.urdf (robot description, URDF)
Before this commit: robot robot, 6 links, 5 joints
Links:
- link Apple: geometry collision box size=3.200977395258038 0.5474678645673197 0.9669883776559041; visual box size=3.200977395258038 0.5474678645673197 0.9669883776559041
- link Dog: geometry collision box size=1.1976653649359406 0.34394622944971753 1.075043933374788; visual box size=1.1976653649359406 0.34394622944971753 1.075043933374788
- link Flower: geometry collision box size=1.670864340962695 0.748583221070344 0.22280470593389534; visual box size=1.670864340962695 0.748583221070344 0.22280470593389534
- link Fox: geometry collision box size=1.829609810625592 1.295121776559723 0.8009665625236799; visual box size=1.829609810625592 1.295121776559723 0.8009665625236799
- link Person: geometry collision box size=0.9731157332047287 1.5994684540345556 1.8797641544929609; visual box size=0.9731157332047287 1.5994684540345556 1.8797641544929609
- link Torso: geometry collision box size=0.2865823664932303 1 1; visual box size=0.2865823664932303 1 1
Joints:
- joint Apple_Dog: origin xyz=3.6573237918235595 0 0 rpy=0 0 0 -> xyz=3.200977395258038 0 0 rpy=0 0 0
- joint Dog_Person: origin xyz=0.5635370020764442 0.8148271582739918 0 rpy=0 0 0 -> xyz=0.5988326824679703 0 0.537521966687394 rpy=0 0 0
- joint Fox_Flower: origin xyz=0 0 0.8647957507309558 rpy=0 0 0 -> xyz=0 0 0.8009665625236799 rpy=0 0 0
- joint Person_Fox: origin xyz=0.6672023068336883 0 0.9258285236595287 rpy=0 0 0 -> xyz=0.48655786660236433 0 0.9398820772464804 rpy=0 0 0
- joint Torso_Apple: origin xyz=0.4203787607110572 0 3 rpy=0 0 0 -> xyz=2.1432911832466153 0 3 rpy=0 0 0

Commit message: now I just have to edit the body and then regenerate

File: body.urdf (robot description, URDF)
Before this commit: robot robot, 6 links, 5 joints
Links:
- added link Lee, mass 1; collision box size=0.5620727029877233 1.6878846418139815 1.3908086874460062; visual box size=0.5620727029877233 1.6878846418139815 1.3908086874460062
- link Apple: geometry collision box size=3.438131869405769 3.7610268486878784 3.126152575450029; visual box size=3.438131869405769 3.7610268486878784 3.126152575450029
- link Dog: geometry collision box size=1.1281782654978796 1.9431274474388012 0.06416467198921749; visual box size=1.1281782654978796 1.9431274474388012 0.06416467198921749
- link Flower: geometry collision box size=0.3367209546825507 1.3486041293976767 1.882796917490526; visual box size=0.3367209546825507 1.3486041293976767 1.882796917490526
- link Fox: geometry collision box size=1.067018111736529 0.21566321243271314 1.168918029164718; visual box size=1.067018111736529 0.21566321243271314 1.168918029164718
- link Person: geometry collision box size=1.8324140523273367 0.7377966616453806 1.6936260565392793; visual box size=1.8324140523273367 0.7377966616453806 1.6936260565392793
- link Torso: geometry collision box size=0.25176690618262754 1 1; visual box size=0.25176690618262754 1 1
Joints:
- added joint Flower_Lee: type revolute, parent Flower, child Lee, origin xyz=0.16836047734127535 0.6743020646988384 0 rpy=0 0 0, axis 0 1 0, limit lower=-3.14159 upper=3.14159 effort=0.0 velocity=0.0
- joint Apple_Dog: origin xyz=3.200977395258038 0 0 rpy=0 0 0 -> xyz=3.438131869405769 0 0 rpy=0 0 0
- joint Dog_Person: origin xyz=0.5988326824679703 0 0.537521966687394 rpy=0 0 0 -> xyz=0.5640891327489398 0 0.032082335994608746 rpy=0 0 0
- joint Fox_Flower: origin xyz=0 0 0.8009665625236799 rpy=0 0 0 -> xyz=1.067018111736529 0 0 rpy=0 0 0
- joint Person_Fox: origin xyz=0.48655786660236433 0 0.9398820772464804 rpy=0 0 0 -> xyz=0.9162070261636683 0 0.8468130282696397 rpy=0 0 0
- joint Torso_Apple: origin xyz=2.1432911832466153 0 3 rpy=0 0 0 -> xyz=0.12588345309131377 0 3 rpy=0 0 0

Commit message: going to try to fix this key error

File: body.urdf (robot description, URDF)
Before this commit: robot robot, 7 links, 6 joints
Links:
- removed link Lee
- link Apple: geometry collision box size=3.6382352049227364 2.9373267310782825 3.2062377149119285; visual box size=3.6382352049227364 2.9373267310782825 3.2062377149119285
- link Dog: geometry collision box size=1.7381652761476019 1.827175986507125 0.284472383896345; visual box size=1.7381652761476019 1.827175986507125 0.284472383896345
- link Flower: geometry collision box size=1.9446240787865843 0.6809254657140362 0.585650756494396; visual box size=1.9446240787865843 0.6809254657140362 0.585650756494396
- link Fox: geometry collision box size=0.1279571947386804 1.3191856408663463 0.9733311339137705; visual box size=0.1279571947386804 1.3191856408663463 0.9733311339137705
- link Person: geometry collision box size=1.117981909865049 0.8085118156231368 0.16764967507398842; visual box size=1.117981909865049 0.8085118156231368 0.16764967507398842
- link Torso: geometry collision box size=1.707322726675308 1 1; visual box size=1.707322726675308 1 1
Joints:
- removed joint Flower_Lee
- joint Apple_Dog: origin xyz=3.438131869405769 0 0 rpy=0 0 0 -> xyz=3.6382352049227364 0 0 rpy=0 0 0
- joint Dog_Person: origin xyz=0.5640891327489398 0 0.032082335994608746 rpy=0 0 0 -> xyz=0.8690826380738009 0.9135879932535625 0 rpy=0 0 0
- joint Fox_Flower: origin xyz=1.067018111736529 0 0 rpy=0 0 0 -> xyz=0 0 0.9733311339137705 rpy=0 0 0
- joint Person_Fox: origin xyz=0.9162070261636683 0 0.8468130282696397 rpy=0 0 0 -> xyz=0.5589909549325245 0 0.08382483753699421 rpy=0 0 0
- joint Torso_Apple: origin xyz=0.12588345309131377 0 3 rpy=0 0 0 -> xyz=2.853661363337654 0 3 rpy=0 0 0
