Commit message: I think I fixed the keyerror

File: body1.urdf (robot description, URDF)
Before this commit: robot robot, 6 links, 5 joints
Links:
- link Apple: geometry collision box size=2.4924185214590695 3.5452802136976094 3.933171102014727; visual box size=2.4924185214590695 3.5452802136976094 3.933171102014727
- link Dog: geometry collision box size=1.0785706187805644 1.9599213674678613 1.1637345532380907; visual box size=1.0785706187805644 1.9599213674678613 1.1637345532380907
- link Flower: geometry collision box size=1.0712612892303137 0.45782283697601933 1.0210344769686435; visual box size=1.0712612892303137 0.45782283697601933 1.0210344769686435
- link Fox: geometry collision box size=0.13956191893637238 0.3263747447060279 1.2877608385299428; visual box size=0.13956191893637238 0.3263747447060279 1.2877608385299428
- link Person: geometry collision box size=0.43604599257139887 1.7082796311673687 1.2849016624579173; visual box size=0.43604599257139887 1.7082796311673687 1.2849016624579173
- link Torso: geometry collision box size=1.9292581502580393 1 1; visual box size=1.9292581502580393 1 1
Joints:
- joint Apple_Dog: origin xyz=3.6382352049227364 0 0 rpy=0 0 0 -> xyz=2.4924185214590695 0 0 rpy=0 0 0
- joint Dog_Person: origin xyz=0.8690826380738009 0.9135879932535625 0 rpy=0 0 0 -> xyz=0.5392853093902822 0 0.5818672766190454 rpy=0 0 0
- joint Fox_Flower: origin xyz=0 0 0.9733311339137705 rpy=0 0 0 -> xyz=0.06978095946818619 0 0.6438804192649714 rpy=0 0 0
- joint Person_Fox: origin xyz=0.5589909549325245 0 0.08382483753699421 rpy=0 0 0 -> xyz=0.21802299628569943 0 0.6424508312289586 rpy=0 0 0
- joint Torso_Apple: origin xyz=2.853661363337654 0 3 rpy=0 0 0 -> xyz=2.96462907512902 0 3 rpy=0 0 0
