Commit message: resized some things

File: body0.urdf (robot description, URDF)
Before this commit: robot robot, 5 links, 4 joints
Links:
- link Aardvark: geometry collision box size=1.4381140383412014 0.42058217158783373 3.1888559909550462; visual box size=1.4381140383412014 0.42058217158783373 3.1888559909550462
- link Abacus: geometry collision box size=1.903237578390486 1.653108331221305 1.2371053272245414; visual box size=1.903237578390486 1.653108331221305 1.2371053272245414
- link Abbey: geometry collision box size=0.7482721384454476 1.953972830574633 1.6244049395465716; visual box size=0.7482721384454476 1.953972830574633 1.6244049395465716
- link Abdomen: geometry collision box size=0.1427137270288088 0.9651986005186723 1.502563484538593; visual box size=0.1427137270288088 0.9651986005186723 1.502563484538593
- link Torso: geometry collision box size=1.2986781460208165 1 1; visual box size=1.2986781460208165 1 1
Joints:
- joint Aardvark_Abacus: origin xyz=2.4416442560895226 0 0 rpy=0 0 0 -> xyz=1.4381140383412014 0 0 rpy=0 0 0
- joint Abacus_Abbey: origin xyz=0.9606932771120097 0.85380904529497 0 rpy=0 0 0 -> xyz=0.951618789195243 0 0.6185526636122707 rpy=0 0 0
- joint Abbey_Abdomen: origin xyz=0 0.1281094076526903 0.51976848175642 rpy=0 0 0 -> xyz=0 0 1.6244049395465716 rpy=0 0 0
- joint Torso_Aardvark: origin xyz=-2.1941499845730528 0 3 rpy=0 0 0 -> xyz=-1.3506609269895917 0 3 rpy=0 0 0

File: body1.urdf (robot description, URDF)
Before this commit: robot robot, 5 links, 4 joints
Links:
- link Aardvark: geometry collision box size=1.4381140383412014 0.42058217158783373 3.1888559909550462; visual box size=1.4381140383412014 0.42058217158783373 3.1888559909550462
- link Abacus: geometry collision box size=1.903237578390486 1.653108331221305 1.2371053272245414; visual box size=1.903237578390486 1.653108331221305 1.2371053272245414
- link Abbey: geometry collision box size=0.7482721384454476 1.953972830574633 1.6244049395465716; visual box size=0.7482721384454476 1.953972830574633 1.6244049395465716
- link Abdomen: geometry collision box size=0.1427137270288088 0.9651986005186723 1.502563484538593; visual box size=0.1427137270288088 0.9651986005186723 1.502563484538593
- link Torso: geometry collision box size=0.01152206800525657 0.2865633480884435 0.42861493303267206; visual box size=0.01152206800525657 0.2865633480884435 0.42861493303267206
Joints:
- joint Aardvark_Abacus: origin xyz=2.4416442560895226 0 0 rpy=0 0 0 -> xyz=1.4381140383412014 0 0 rpy=0 0 0
- joint Abacus_Abbey: origin xyz=0.9606932771120097 0.85380904529497 0 rpy=0 0 0 -> xyz=0.951618789195243 0 0.6185526636122707 rpy=0 0 0
- joint Abbey_Abdomen: origin xyz=0 0.1281094076526903 0.51976848175642 rpy=0 0 0 -> xyz=0 0 1.6244049395465716 rpy=0 0 0
- joint Torso_Aardvark: origin xyz=-2.1941499845730528 0 3 rpy=0 0 0 -> xyz=-1.3506609269895917 0 3 rpy=0 0 0

Commit message: fixed wrong fitness getting added to array

File: body0.urdf (robot description, URDF)
Before this commit: robot robot, 5 links, 4 joints
Links:
- link Aardvark: geometry collision box size=1.6510696907310258 3.9051827012685627 0.44921450114819184; visual box size=1.6510696907310258 3.9051827012685627 0.44921450114819184
- link Abacus: geometry collision box size=1.1016226429326075 0.011884031847990695 0.481609620632524; visual box size=1.1016226429326075 0.011884031847990695 0.481609620632524
- link Abbey: geometry collision box size=1.0973729317409209 1.050565206866036 0.290377121241576; visual box size=1.0973729317409209 1.050565206866036 0.290377121241576
- link Abdomen: geometry collision box size=1.1970028597741522 1.1316320086533787 0.7685144643863813; visual box size=1.1970028597741522 1.1316320086533787 0.7685144643863813
- link Torso: geometry collision box size=0.3850097507299921 1 1; visual box size=0.3850097507299921 1 1
Joints:
- joint Aardvark_Abacus: origin xyz=1.4381140383412014 0 0 rpy=0 0 0 -> xyz=1.6510696907310258 0 0 rpy=0 0 0
- joint Abacus_Abbey: origin xyz=0.951618789195243 0 0.6185526636122707 rpy=0 0 0 -> xyz=0.5508113214663037 0 0.240804810316262 rpy=0 0 0
- joint Abbey_Abdomen: origin xyz=0 0 1.6244049395465716 rpy=0 0 0 -> xyz=0.5486864658704604 0 0.145188560620788 rpy=0 0 0
- joint Torso_Aardvark: origin xyz=-1.3506609269895917 0 3 rpy=0 0 0 -> xyz=2.192504875364996 0 3 rpy=0 0 0

File: body2.urdf (robot description, URDF)
Before this commit: robot robot, 5 links, 4 joints
Links:
- link Aardvark: geometry collision box size=0.4627453260818224 1.5094529238216174 3.427191385179227; visual box size=0.4627453260818224 1.5094529238216174 3.427191385179227
- link Abacus: geometry collision box size=0.7069241289030193 1.1793793389879248 0.991952428459105; visual box size=0.7069241289030193 1.1793793389879248 0.991952428459105
- link Abbey: geometry collision box size=1.9853043799658694 1.5693253721110227 0.38588348627879254; visual box size=1.9853043799658694 1.5693253721110227 0.38588348627879254
- link Abdomen: geometry collision box size=1.4341821290919081 1.8761598122709557 1.6456432044577827; visual box size=1.4341821290919081 1.8761598122709557 1.6456432044577827
- link Torso: geometry collision box size=1.4535010034857498 0.8676659165453238 1.1548866383275107; visual box size=1.4535010034857498 0.8676659165453238 1.1548866383275107
Joints:
- joint Aardvark_Abacus: origin xyz=1.6510696907310258 0 0 rpy=0 0 0 -> xyz=0.4627453260818224 0 0 rpy=0 0 0
- joint Abacus_Abbey: origin xyz=0.5508113214663037 0 0.240804810316262 rpy=0 0 0 -> xyz=0.3534620644515096 0 0.4959762142295525 rpy=0 0 0
- joint Abbey_Abdomen: origin xyz=0.5486864658704604 0 0.145188560620788 rpy=0 0 0 -> xyz=0 0 0.38588348627879254 rpy=0 0 0
- joint Torso_Aardvark: origin xyz=2.192504875364996 0 3 rpy=0 0 0 -> xyz=-0.9816605184270498 0 3 rpy=0 0 0

File: body3.urdf (robot description, URDF)
Before this commit: robot robot, 5 links, 4 joints
Links:
- link Aardvark: geometry collision box size=0.4627453260818224 1.5094529238216174 3.427191385179227; visual box size=0.4627453260818224 1.5094529238216174 3.427191385179227
- link Abacus: geometry collision box size=0.7069241289030193 1.1793793389879248 0.991952428459105; visual box size=0.7069241289030193 1.1793793389879248 0.991952428459105
- link Abbey: geometry collision box size=1.9853043799658694 1.5693253721110227 0.38588348627879254; visual box size=1.9853043799658694 1.5693253721110227 0.38588348627879254
- link Abdomen: geometry collision box size=1.4341821290919081 1.8761598122709557 1.6456432044577827; visual box size=1.4341821290919081 1.8761598122709557 1.6456432044577827
- link Torso: geometry collision box size=0.11890612283212176 1.4859809163323625 1.9837054816009778; visual box size=0.11890612283212176 1.4859809163323625 1.9837054816009778
Joints:
- joint Aardvark_Abacus: origin xyz=1.6510696907310258 0 0 rpy=0 0 0 -> xyz=0.4627453260818224 0 0 rpy=0 0 0
- joint Abacus_Abbey: origin xyz=0.5508113214663037 0 0.240804810316262 rpy=0 0 0 -> xyz=0.3534620644515096 0 0.4959762142295525 rpy=0 0 0
- joint Abbey_Abdomen: origin xyz=0.5486864658704604 0 0.145188560620788 rpy=0 0 0 -> xyz=0 0 0.38588348627879254 rpy=0 0 0
- joint Torso_Aardvark: origin xyz=2.192504875364996 0 3 rpy=0 0 0 -> xyz=-0.9816605184270498 0 3 rpy=0 0 0

File: body4.urdf (robot description, URDF)
Before this commit: robot robot, 5 links, 4 joints
Links:
- link Aardvark: geometry collision box size=0.4627453260818224 1.5094529238216174 3.427191385179227; visual box size=0.4627453260818224 1.5094529238216174 3.427191385179227
- link Abacus: geometry collision box size=0.7069241289030193 1.1793793389879248 0.991952428459105; visual box size=0.7069241289030193 1.1793793389879248 0.991952428459105
- link Abbey: geometry collision box size=1.9853043799658694 1.5693253721110227 0.38588348627879254; visual box size=1.9853043799658694 1.5693253721110227 0.38588348627879254
- link Abdomen: geometry collision box size=1.4341821290919081 1.8761598122709557 1.6456432044577827; visual box size=1.4341821290919081 1.8761598122709557 1.6456432044577827
- link Torso: geometry collision box size=1.8367605267102949 1.018992422042723 1.5132352854732123; visual box size=1.8367605267102949 1.018992422042723 1.5132352854732123
Joints:
- joint Aardvark_Abacus: origin xyz=1.6510696907310258 0 0 rpy=0 0 0 -> xyz=0.4627453260818224 0 0 rpy=0 0 0
- joint Abacus_Abbey: origin xyz=0.5508113214663037 0 0.240804810316262 rpy=0 0 0 -> xyz=0.3534620644515096 0 0.4959762142295525 rpy=0 0 0
- joint Abbey_Abdomen: origin xyz=0.5486864658704604 0 0.145188560620788 rpy=0 0 0 -> xyz=0 0 0.38588348627879254 rpy=0 0 0
- joint Torso_Aardvark: origin xyz=2.192504875364996 0 3 rpy=0 0 0 -> xyz=-0.9816605184270498 0 3 rpy=0 0 0

File: body5.urdf (robot description, URDF)
Before this commit: robot robot, 5 links, 4 joints
Links:
- link Aardvark: geometry collision box size=0.6270328287730824 0.08962853636233303 0.07417319373955866; visual box size=0.6270328287730824 0.08962853636233303 0.07417319373955866
- link Abacus: geometry collision box size=0.7901424532921679 0.3200411760598658 1.7354823622147495; visual box size=0.7901424532921679 0.3200411760598658 1.7354823622147495
- link Abbey: geometry collision box size=1.3972364917198317 0.5111781921749856 1.3393954401029113; visual box size=1.3972364917198317 0.5111781921749856 1.3393954401029113
- link Abdomen: geometry collision box size=1.5890504990343906 1.29328723900446 1.3550236345521927; visual box size=1.5890504990343906 1.29328723900446 1.3550236345521927
- link Torso: geometry collision box size=0.3448317697686145 0.8951479384410852 1.356132641466123; visual box size=0.3448317697686145 0.8951479384410852 1.356132641466123
Joints:
- joint Aardvark_Abacus: origin xyz=1.6510696907310258 0 0 rpy=0 0 0 -> xyz=0.6270328287730824 0 0 rpy=0 0 0
- joint Abacus_Abbey: origin xyz=0.5508113214663037 0 0.240804810316262 rpy=0 0 0 -> xyz=0 0 1.7354823622147495 rpy=0 0 0
- joint Abbey_Abdomen: origin xyz=0.5486864658704604 0 0.145188560620788 rpy=0 0 0 -> xyz=0 0.2555890960874928 0.6696977200514557 rpy=0 0 0
- joint Torso_Aardvark: origin xyz=2.192504875364996 0 3 rpy=0 0 0 -> xyz=3.0896455066890964 0 3 rpy=0 0 0

Commit message: fixed mutation errors

File: body0.urdf (robot description, URDF)
Before this commit: robot robot, 5 links, 4 joints
Links:
- link Aardvark: geometry collision box size=3.99451813506449 0.33022897870306345 3.819542917285506; visual box size=3.99451813506449 0.33022897870306345 3.819542917285506
- link Abacus: geometry collision box size=1.6408123667862005 0.8871659894909432 1.934348093062511; visual box size=1.6408123667862005 0.8871659894909432 1.934348093062511
- link Abbey: geometry collision box size=0.7186072819632405 0.6379090628561577 1.283332443388848; visual box size=0.7186072819632405 0.6379090628561577 1.283332443388848
- link Abdomen: geometry collision box size=0.6996751078101597 0.18247107222318926 0.34926632799061963; visual box size=0.6996751078101597 0.18247107222318926 0.34926632799061963
- link Torso: geometry collision box size=1.356436592916205 1 1; visual box size=1.356436592916205 1 1
Joints:
- joint Aardvark_Abacus: origin xyz=1.6510696907310258 0 0 rpy=0 0 0 -> xyz=3.99451813506449 0 0 rpy=0 0 0
- joint Abacus_Abbey: origin xyz=0.5508113214663037 0 0.240804810316262 rpy=0 0 0 -> xyz=0 0 1.934348093062511 rpy=0 0 0
- joint Abbey_Abdomen: origin xyz=0.5486864658704604 0 0.145188560620788 rpy=0 0 0 -> xyz=0 0 1.283332443388848 rpy=0 0 0
- joint Torso_Aardvark: origin xyz=2.192504875364996 0 3 rpy=0 0 0 -> xyz=1.6782182964581025 0 3 rpy=0 0 0

File: body1.urdf (robot description, URDF)
Before this commit: robot robot, 5 links, 4 joints
Links:
- link Aardvark: geometry collision box size=3.99451813506449 0.33022897870306345 3.819542917285506; visual box size=3.99451813506449 0.33022897870306345 3.819542917285506
- link Abacus: geometry collision box size=1.6408123667862005 0.8871659894909432 1.934348093062511; visual box size=1.6408123667862005 0.8871659894909432 1.934348093062511
- link Abbey: geometry collision box size=0.7186072819632405 0.6379090628561577 1.283332443388848; visual box size=0.7186072819632405 0.6379090628561577 1.283332443388848
- link Abdomen: geometry collision box size=0.6996751078101597 0.18247107222318926 0.34926632799061963; visual box size=0.6996751078101597 0.18247107222318926 0.34926632799061963
- link Torso: geometry collision box size=0.8334764083608481 0.6391732276155957 1.9695049456857745; visual box size=0.8334764083608481 0.6391732276155957 1.9695049456857745
Joints:
- joint Aardvark_Abacus: origin xyz=1.6510696907310258 0 0 rpy=0 0 0 -> xyz=3.99451813506449 0 0 rpy=0 0 0
- joint Abacus_Abbey: origin xyz=0.5508113214663037 0 0.240804810316262 rpy=0 0 0 -> xyz=0 0 1.934348093062511 rpy=0 0 0
- joint Abbey_Abdomen: origin xyz=0.5486864658704604 0 0.145188560620788 rpy=0 0 0 -> xyz=0 0 1.283332443388848 rpy=0 0 0
- joint Torso_Aardvark: origin xyz=2.192504875364996 0 3 rpy=0 0 0 -> xyz=1.6782182964581025 0 3 rpy=0 0 0

Commit message: added functionallity to be able replay past simulations

File: body0.urdf (robot description, URDF)
Before this commit: robot robot, 5 links, 4 joints
Links:
- link Aardvark: geometry collision box size=3.9363384728317157 0.13696371380342853 1.6518209906137868; visual box size=3.9363384728317157 0.13696371380342853 1.6518209906137868
- link Abacus: geometry collision box size=0.2746270597477265 0.8162073829157213 1.9651243824528073; visual box size=0.2746270597477265 0.8162073829157213 1.9651243824528073
- link Abbey: geometry collision box size=1.821151693595726 1.288966503280712 0.6348665639125157; visual box size=1.821151693595726 1.288966503280712 0.6348665639125157
- link Abdomen: geometry collision box size=1.5181804617821253 1.7314448215940077 0.7845046480229252; visual box size=1.5181804617821253 1.7314448215940077 0.7845046480229252
- link Torso: geometry collision box size=0.8945425233484918 1 1; visual box size=0.8945425233484918 1 1
Joints:
- joint Aardvark_Abacus: origin xyz=3.99451813506449 0 0 rpy=0 0 0 -> xyz=3.9363384728317157 0 0 rpy=0 0 0
- joint Abacus_Abbey: origin xyz=0 0 1.934348093062511 rpy=0 0 0 -> xyz=0.13731352987386325 0 0.9825621912264036 rpy=0 0 0
- joint Abbey_Abdomen: origin xyz=0 0 1.283332443388848 rpy=0 0 0 -> xyz=0.910575846797863 0 0.31743328195625786 rpy=0 0 0
- joint Torso_Aardvark: origin xyz=1.6782182964581025 0 3 rpy=0 0 0 -> xyz=-1.552728738325754 0 3 rpy=0 0 0

File: body1.urdf (robot description, URDF)
Before this commit: robot robot, 5 links, 4 joints
Links:
- link Aardvark: geometry collision box size=3.9363384728317157 0.13696371380342853 1.6518209906137868; visual box size=3.9363384728317157 0.13696371380342853 1.6518209906137868
- link Abacus: geometry collision box size=0.2746270597477265 0.8162073829157213 1.9651243824528073; visual box size=0.2746270597477265 0.8162073829157213 1.9651243824528073
- link Abbey: geometry collision box size=1.821151693595726 1.288966503280712 0.6348665639125157; visual box size=1.821151693595726 1.288966503280712 0.6348665639125157
- link Abdomen: geometry collision box size=1.5181804617821253 1.7314448215940077 0.7845046480229252; visual box size=1.5181804617821253 1.7314448215940077 0.7845046480229252
- link Torso: geometry collision box size=0.5315885122090345 1.856482849275269 0.8012767000097856; visual box size=0.5315885122090345 1.856482849275269 0.8012767000097856
Joints:
- joint Aardvark_Abacus: origin xyz=3.99451813506449 0 0 rpy=0 0 0 -> xyz=3.9363384728317157 0 0 rpy=0 0 0
- joint Abacus_Abbey: origin xyz=0 0 1.934348093062511 rpy=0 0 0 -> xyz=0.13731352987386325 0 0.9825621912264036 rpy=0 0 0
- joint Abbey_Abdomen: origin xyz=0 0 1.283332443388848 rpy=0 0 0 -> xyz=0.910575846797863 0 0.31743328195625786 rpy=0 0 0
- joint Torso_Aardvark: origin xyz=1.6782182964581025 0 3 rpy=0 0 0 -> xyz=-1.552728738325754 0 3 rpy=0 0 0
