Commit message: refactored the files so that each file from each generation gets saved, broke replaying simulations

File: 2_body2.urdf (robot description, URDF)
Before this commit: robot robot, 5 links, 4 joints
Links:
- link Aardvark: geometry collision box size=0.8443523151444023 2.3690339071314224 3.615170599662533; visual box size=0.8443523151444023 2.3690339071314224 3.615170599662533
- link Abacus: geometry collision box size=1.653919558759366 1.295097747701477 0.78461660577212; visual box size=1.653919558759366 1.295097747701477 0.78461660577212
- link Abbey: geometry collision box size=1.9993100256060272 1.6687598371184182 1.0277132480372164; visual box size=1.9993100256060272 1.6687598371184182 1.0277132480372164
- link Abdomen: geometry collision box size=1.14607481018203 0.736380899740408 0.06871905803835188; visual box size=1.14607481018203 0.736380899740408 0.06871905803835188
- link Torso: geometry collision box size=1.8804590421565284 1.2351956191471642 1.9002523611068225; visual box size=1.8804590421565284 1.2351956191471642 1.9002523611068225
Joints:
- joint Aardvark_Abacus: origin xyz=3.9363384728317157 0 0 rpy=0 0 0 -> xyz=0.8443523151444023 0 0 rpy=0 0 0
- joint Abacus_Abbey: origin xyz=0.13731352987386325 0 0.9825621912264036 rpy=0 0 0 -> xyz=0.826959779379683 0.6475488738507384 0 rpy=0 0 0
- joint Abbey_Abdomen: origin xyz=0.910575846797863 0 0.31743328195625786 rpy=0 0 0 -> xyz=0.9996550128030136 0 0.5138566240186082 rpy=0 0 0
- joint Torso_Aardvark: origin xyz=-1.552728738325754 0 3 rpy=0 0 0 -> xyz=-3.019760338572925 0 3 rpy=0 0 0
