Commit message: added some new diagrams

File: 0_body0.urdf (robot description, URDF)
Before this commit: robot robot, 5 links, 4 joints
Links:
- link Aardvark: geometry collision box size=3.809831876702445 3.384726543936776 0.888054231997037; visual box size=3.809831876702445 3.384726543936776 0.888054231997037
- link Abacus: geometry collision box size=1.6179804663272213 1.40299829758463 1.8524473309548843; visual box size=1.6179804663272213 1.40299829758463 1.8524473309548843
- link Abbey: geometry collision box size=1.5962836585062163 1.1330807153228497 1.5064179736926249; visual box size=1.5962836585062163 1.1330807153228497 1.5064179736926249
- link Abdomen: geometry collision box size=1.3415052800795448 1.1025877178413377 0.4958928691200064; visual box size=1.3415052800795448 1.1025877178413377 0.4958928691200064
- link Torso: geometry collision box size=0.2027929345532573 1 1; visual box size=0.2027929345532573 1 1
Joints:
- joint Aardvark_Abacus: origin xyz=3.342621851514235 0 0 rpy=0 0 0 -> xyz=3.809831876702445 0 0 rpy=0 0 0
- joint Abacus_Abbey: origin xyz=0 0 1.2872973886024495 rpy=0 0 0 -> xyz=0 0.701499148792315 0.9262236654774422 rpy=0 0 0
- joint Abbey_Abdomen: origin xyz=0 0 1.663721641610068 rpy=0 0 0 -> xyz=0 0.5665403576614249 0.7532089868463124 rpy=0 0 0
- joint Torso_Aardvark: origin xyz=-2.2381693067671784 0 3 rpy=0 0 0 -> xyz=-1.8986035327233712 0 3 rpy=0 0 0

File: 1_body0.urdf (robot description, URDF)
Before this commit: robot robot, 5 links, 4 joints
Links:
- link Aardvark: geometry collision box size=3.809831876702445 3.384726543936776 0.888054231997037; visual box size=3.809831876702445 3.384726543936776 0.888054231997037
- link Abacus: geometry collision box size=1.6179804663272213 1.40299829758463 1.8524473309548843; visual box size=1.6179804663272213 1.40299829758463 1.8524473309548843
- link Abbey: geometry collision box size=1.5962836585062163 1.1330807153228497 1.5064179736926249; visual box size=1.5962836585062163 1.1330807153228497 1.5064179736926249
- link Abdomen: geometry collision box size=1.3415052800795448 1.1025877178413377 0.4958928691200064; visual box size=1.3415052800795448 1.1025877178413377 0.4958928691200064
- link Torso: geometry collision box size=0.2027929345532573 1 1; visual box size=0.2027929345532573 1 1
Joints:
- joint Aardvark_Abacus: origin xyz=3.342621851514235 0 0 rpy=0 0 0 -> xyz=3.809831876702445 0 0 rpy=0 0 0
- joint Abacus_Abbey: origin xyz=0 0 1.2872973886024495 rpy=0 0 0 -> xyz=0 0.701499148792315 0.9262236654774422 rpy=0 0 0
- joint Abbey_Abdomen: origin xyz=0 0 1.663721641610068 rpy=0 0 0 -> xyz=0 0.5665403576614249 0.7532089868463124 rpy=0 0 0
- joint Torso_Aardvark: origin xyz=-2.2381693067671784 0 3 rpy=0 0 0 -> xyz=-1.8986035327233712 0 3 rpy=0 0 0

File: 1_body1.urdf (robot description, URDF)
Before this commit: robot robot, 5 links, 4 joints
Links:
- link Aardvark: geometry collision box size=3.809831876702445 3.384726543936776 0.888054231997037; visual box size=3.809831876702445 3.384726543936776 0.888054231997037
- link Abacus: geometry collision box size=1.6179804663272213 1.40299829758463 1.8524473309548843; visual box size=1.6179804663272213 1.40299829758463 1.8524473309548843
- link Abbey: geometry collision box size=1.5962836585062163 1.1330807153228497 1.5064179736926249; visual box size=1.5962836585062163 1.1330807153228497 1.5064179736926249
- link Abdomen: geometry collision box size=1.3415052800795448 1.1025877178413377 0.4958928691200064; visual box size=1.3415052800795448 1.1025877178413377 0.4958928691200064
- link Torso: geometry collision box size=1.262517920188162 1.6853747487981234 0.5501271134408041; visual box size=1.262517920188162 1.6853747487981234 0.5501271134408041
Joints:
- joint Aardvark_Abacus: origin xyz=3.342621851514235 0 0 rpy=0 0 0 -> xyz=3.809831876702445 0 0 rpy=0 0 0
- joint Abacus_Abbey: origin xyz=0 0 1.2872973886024495 rpy=0 0 0 -> xyz=0 0.701499148792315 0.9262236654774422 rpy=0 0 0
- joint Abbey_Abdomen: origin xyz=0 0 1.663721641610068 rpy=0 0 0 -> xyz=0 0.5665403576614249 0.7532089868463124 rpy=0 0 0
- joint Torso_Aardvark: origin xyz=-2.2381693067671784 0 3 rpy=0 0 0 -> xyz=-1.8986035327233712 0 3 rpy=0 0 0

File: 1_body2.urdf (robot description, URDF)
Before this commit: robot robot, 5 links, 4 joints
Links:
- link Aardvark: geometry collision box size=3.96938755340077 3.2425597422002794 3.3508371320994774; visual box size=3.96938755340077 3.2425597422002794 3.3508371320994774
- link Abacus: geometry collision box size=0.2148651065815108 1.212823425741917 0.11015538309152029; visual box size=0.2148651065815108 1.212823425741917 0.11015538309152029
- link Abbey: geometry collision box size=0.12764032050554097 1.5703036325099828 1.3597181528679774; visual box size=0.12764032050554097 1.5703036325099828 1.3597181528679774
- link Abdomen: geometry collision box size=0.7765904757086541 0.810505829783126 1.1685743403284616; visual box size=0.7765904757086541 0.810505829783126 1.1685743403284616
- link Torso: geometry collision box size=1.6428428998078402 0.5800613178546254 0.9251142982879201; visual box size=1.6428428998078402 0.5800613178546254 0.9251142982879201
Joints:
- joint Aardvark_Abacus: origin xyz=3.5020623390555397 0 0 rpy=0 0 0 -> xyz=3.96938755340077 0 0 rpy=0 0 0
- joint Abacus_Abbey: origin xyz=0.6014067280289621 0.5273936523433227 0 rpy=0 0 0 -> xyz=0.1074325532907554 0 0.055077691545760143 rpy=0 0 0
- joint Abbey_Abdomen: origin xyz=1.1712727029226304 0 0 rpy=0 0 0 -> xyz=0.06382016025277049 0 0.6798590764339887 rpy=0 0 0
- joint Torso_Aardvark: origin xyz=-2.0453293105402386 0 3 rpy=0 0 0 -> xyz=3.147915786386704 0 3 rpy=0 0 0

File: 2_body1.urdf (robot description, URDF)
Before this commit: robot robot, 5 links, 4 joints
Links:
- link Aardvark: geometry collision box size=3.809831876702445 3.384726543936776 0.888054231997037; visual box size=3.809831876702445 3.384726543936776 0.888054231997037
- link Abacus: geometry collision box size=1.6179804663272213 1.40299829758463 1.8524473309548843; visual box size=1.6179804663272213 1.40299829758463 1.8524473309548843
- link Abbey: geometry collision box size=1.5962836585062163 1.1330807153228497 1.5064179736926249; visual box size=1.5962836585062163 1.1330807153228497 1.5064179736926249
- link Abdomen: geometry collision box size=1.3415052800795448 1.1025877178413377 0.4958928691200064; visual box size=1.3415052800795448 1.1025877178413377 0.4958928691200064
- link Torso: geometry collision box size=0.8959364297327295 0.638197175543695 1.9853787887448124; visual box size=0.8959364297327295 0.638197175543695 1.9853787887448124
Joints:
- joint Aardvark_Abacus: origin xyz=3.96938755340077 0 0 rpy=0 0 0 -> xyz=3.809831876702445 0 0 rpy=0 0 0
- joint Abacus_Abbey: origin xyz=0.1074325532907554 0 0.055077691545760143 rpy=0 0 0 -> xyz=0 0.701499148792315 0.9262236654774422 rpy=0 0 0
- joint Abbey_Abdomen: origin xyz=0.06382016025277049 0 0.6798590764339887 rpy=0 0 0 -> xyz=0 0.5665403576614249 0.7532089868463124 rpy=0 0 0
- joint Torso_Aardvark: origin xyz=3.147915786386704 0 3 rpy=0 0 0 -> xyz=-1.8986035327233712 0 3 rpy=0 0 0

File: 2_body3.urdf (robot description, URDF)
Before this commit: robot robot, 5 links, 4 joints
Links:
- link Aardvark: geometry collision box size=3.96938755340077 3.2425597422002794 3.3508371320994774; visual box size=3.96938755340077 3.2425597422002794 3.3508371320994774
- link Abacus: geometry collision box size=0.2148651065815108 1.212823425741917 0.11015538309152029; visual box size=0.2148651065815108 1.212823425741917 0.11015538309152029
- link Abbey: geometry collision box size=0.12764032050554097 1.5703036325099828 1.3597181528679774; visual box size=0.12764032050554097 1.5703036325099828 1.3597181528679774
- link Abdomen: geometry collision box size=0.7765904757086541 0.810505829783126 1.1685743403284616; visual box size=0.7765904757086541 0.810505829783126 1.1685743403284616
- link Torso: geometry collision box size=0.05505421512989561 1.7348725940964973 0.07368004674374729; visual box size=0.05505421512989561 1.7348725940964973 0.07368004674374729
Joints:
- joint Aardvark_Abacus: origin xyz=3.5020623390555397 0 0 rpy=0 0 0 -> xyz=3.96938755340077 0 0 rpy=0 0 0
- joint Abacus_Abbey: origin xyz=0.6014067280289621 0.5273936523433227 0 rpy=0 0 0 -> xyz=0.1074325532907554 0 0.055077691545760143 rpy=0 0 0
- joint Abbey_Abdomen: origin xyz=1.1712727029226304 0 0 rpy=0 0 0 -> xyz=0.06382016025277049 0 0.6798590764339887 rpy=0 0 0
- joint Torso_Aardvark: origin xyz=-2.0453293105402386 0 3 rpy=0 0 0 -> xyz=3.147915786386704 0 3 rpy=0 0 0
